File: hardware/ADC7177M1/Power.kicad_sch (KiCad schematic)
At the start: 1 part, among them U10 ADR1399KEZ

Commit message: Schematic
Parts:
- removed U10: ADR1399KEZ, Package_LCC:Analog_LCC-8_5x5mm_P1.27mm, symbol Reference_Voltage:ADR1399KEZ
Changed lines of the file:
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@@
 	(paper "A4")
 	(symbol
-		(lib_id "Reference_Voltage:ADR1399KEZ")
-		(at 64.77 87.63 0)
+		(lib_id "power:+5VD")
+		(at 60.96 80.01 0)
 		(unit 1)
 		(exclude_from_sim no)
@@
 		(dnp no)
 		(fields_autoplaced yes)
-		(property "Reference" "U10"
-			(at 69.85 86.3599 0)
-			(effects
-				(font
-					(size 1.27 1.27)
-				)
-				(justify left)
-			)
-		)
-		(property "Value" "ADR1399KEZ"
-			(at 69.85 88.8999 0)
-			(effects
-				(font
-					(size 1.27 1.27)
-				)
-				(justify left)
-			)
-		)
-		(property "Footprint" "Package_LCC:Analog_LCC-8_5x5mm_P1.27mm"
-			(at 64.77 94.615 0)
+		(property "Reference" "#PWR091"
+			(at 60.96 83.82 0)
 			(effects
 				(font
@@
 			)
 		)
-		(property "Datasheet" "https://www.analog.com/media/en/technical-documentation/data-sheets/adr1399.pdf"
-			(at 64.77 96.52 0)
+		(property "Value" "+5VD"
+			(at 60.96 74.93 0)
+			(effects
+				(font
+					(size 1.27 1.27)
+				)
+			)
+		)
+		(property "Footprint" ""
+			(at 60.96 80.01 0)
 			(effects
 				(font
@@
 			)
 		)
-		(property "Description" "Oven-Compensated, Buried Zener, 7.05 V Voltage Reference, LCC-8"
-			(at 64.77 87.63 0)
+		(property "Datasheet" ""
+			(at 60.96 80.01 0)
 			(effects
 				(font
@@
 			)
 		)
-		(pin "6"
-		)
-		(pin "3"
-		)
-		(pin "2"
-		)
-		(pin "5"
-		)
-		(pin "4"
+		(property "Description" "Power symbol creates a global label with name \"+5VD\""
+			(at 60.96 80.01 0)
+			(effects
+				(font
+					(size 1.27 1.27)
+				)
+				(hide yes)
+			)
 		)
 		(pin "1"
-		)
-		(pin "7"
-		)
-		(pin "8"
 		)
 		(instances
 			(project ""
 				(path "/e30159e7-fecb-4b08-a9fd-8c0b6565f013/e382cca3-340a-4115-b733-1d21769b9a67/40ee723a-4bed-42db-bfa8-bbbbb28f1aea"
-					(reference "U10")
+					(reference "#PWR091")
 					(unit 1)
 				)

Commit message: Schematic
Changed lines of the file:
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@@
 	(paper "A4")
 	(symbol
-		(lib_id "power:+5VD")
-		(at 60.96 80.01 0)
+		(lib_id "power:PWR_FLAG")
+		(at 25.4 177.8 180)
+		(unit 1)
+		(exclude_from_sim no)
+		(in_bom yes)
+		(on_board yes)
+		(dnp no)
+		(fields_autoplaced yes)
+		(property "Reference" "#FLG01"
+			(at 25.4 179.705 0)
+			(effects
+				(font
+					(size 1.27 1.27)
+				)
+				(hide yes)
+			)
+		)
+		(property "Value" "PWR_FLAG"
+			(at 25.4 182.88 0)
+			(effects
+				(font
+					(size 1.27 1.27)
+				)
+			)
+		)
+		(property "Footprint" ""
+			(at 25.4 177.8 0)
+			(effects
+				(font
+					(size 1.27 1.27)
+				)
+				(hide yes)
+			)
+		)
+		(property "Datasheet" "~"
+			(at 25.4 177.8 0)
+			(effects
+				(font
+					(size 1.27 1.27)
+				)
+				(hide yes)
+			)
+		)
+		(property "Description" "Special symbol for telling ERC where power comes from"
+			(at 25.4 177.8 0)
+			(effects
+				(font
+					(size 1.27 1.27)
+				)
+				(hide yes)
+			)
+		)
+		(pin "1"
+		)
+		(instances
+			(project ""
+				(path "/e30159e7-fecb-4b08-a9fd-8c0b6565f013/e382cca3-340a-4115-b733-1d21769b9a67/40ee723a-4bed-42db-bfa8-bbbbb28f1aea"
+					(reference "#FLG01")
+					(unit 1)
+				)
+			)
+		)
+	)
+	(symbol
+		(lib_id "power:+15V")
+		(at 25.4 177.8 0)
 		(unit 1)
 		(exclude_from_sim no)
@@
 		(fields_autoplaced yes)
 		(property "Reference" "#PWR091"
-			(at 60.96 83.82 0)
+			(at 25.4 181.61 0)
 			(effects
 				(font
@@
 			)
 		)
-		(property "Value" "+5VD"
-			(at 60.96 74.93 0)
+		(property "Value" "+15V"
+			(at 25.4 172.72 0)
 			(effects
 				(font
@@
 		)
 		(property "Footprint" ""
-			(at 60.96 80.01 0)
+			(at 25.4 177.8 0)
 			(effects
 				(font
@@
 		)
 		(property "Datasheet" ""
-			(at 60.96 80.01 0)
+			(at 25.4 177.8 0)
 			(effects
 				(font
@@
 			)
 		)
-		(property "Description" "Power symbol creates a global label with name \"+5VD\""
-			(at 60.96 80.01 0)
+		(property "Description" "Power symbol creates a global label with name \"+15V\""
+			(at 25.4 177.8 0)
 			(effects
 				(font

Commit message: Schematic and PCB
Parts:
- added C23, C24, C25, C26, C55, C56: 10u, Capacitor_SMD:C_0805_2012Metric, symbol Device:C
- added R27, R29, R50: R, Resistor_SMD:R_0603_1608Metric, symbol Device:R
- added R28, R30, R51: 10k/0.1%, Resistor_SMD:R_0603_1608Metric, symbol Device:R
- added U10: ADP7182ACPZN, Package_CSP:LFCSP-6-1EP_2x2mm_P0.65mm_EP1x1.6mm, symbol ADC7177M1:ADP7182ACPZN
- added U8, U9: ADP7118ACPZN, Package_CSP:LFCSP-6-1EP_2x2mm_P0.65mm_EP1x1.6mm, symbol Regulator_Linear:ADP7118ACPZN
Connections:
- net +15V: now also C24.1, U9.4 (EN), U9.6 (VIN)
- new net: R27.2, R28.1, U8.2 (SENSE/ADJ)
- new net: R50.2, R51.1, U10.2 (ADJ)
- new net: R29.2, R30.1, U9.2 (SENSE/ADJ)
- new net +3.3V: C25.1, R27.1, U8.1 (VOUT)
- new net +5VD: C23.1, U8.4 (EN), U8.6 (VIN)
- new net +7.5V: C26.1, R29.1, U9.1 (VOUT)
- new net -15V: C55.1, U10.3 (EN), U10.6 (VIN), U10.7 (EP)
- new net -2V5: C56.1, R50.1, U10.1 (VOUT)
- new net GNDA: C23.2, C24.2, C25.2, C26.2, C55.2, C56.2, R28.2, R30.2, R51.2, U10.5 (GND), U8.3 (GND), U8.7 (GND), U9.3 (GND), U9.7 (GND)
- no-connect marks 0 -> 2

Commit message: Schematic and PCB
Parts:
- renumbered C25 to C24, C24 to C25, C55 to C27, C56 to C28, R50 to R31, R51 to R32
