File: hardware/ADC7177M1/ADC.kicad_sch (KiCad schematic)
At the start: 13 parts, among them U8 ADA4522-2ARMZ, U9 AD8066ARMZ

Commit message: Schematic
Parts:
- added C35, C37: 1u, Capacitor_SMD:C_0603_1608Metric, symbol Device:C
- added C36, C38, C39, C40, C43, C45, C47, C49: 100n, Capacitor_SMD:C_0603_1608Metric, symbol Device:C
- added C41, C44, C50: 10u, Capacitor_SMD:C_0603_1608Metric, symbol Device:C
- added C42, C46, C48: NFM21PC225B0J3, symbol Device:C_Feedthrough
- added FB1: BLM18HE102SN1, symbol Device:FerriteBead_Small
- added R43, R44: 10k, symbol Device:R
- added R45: 0, symbol Device:R
- added U14: AD7177-2BRUZ, Package_SO:TSSOP-24_4.4x7.8mm_P0.65mm, symbol ADC7177M1:AD7177-2BRUZ
- added Y1: ECS-2520MV-160-BL-TR, Oscillator:Oscillator_SMD_ECS_2520MV-xxx-xx-4Pin_2.5x2.0mm, symbol Oscillator:ECS-2520MV-xxx-xx
- C23: renamed from C28; footprint (none) -> Capacitor_SMD:C_0603_1608Metric
- C24: renamed from C26; footprint (none) -> Capacitor_SMD:C_0603_1608Metric
- C25: renamed from C23; footprint (none) -> Capacitor_SMD:C_0603_1608Metric
- C26: renamed from C24; footprint (none) -> Capacitor_SMD:C_0603_1608Metric
- C27: footprint (none) -> Capacitor_SMD:C_0603_1608Metric
- C28: renamed from C25; footprint (none) -> Capacitor_SMD:C_0603_1608Metric
- R27: renamed from R31; footprint (none) -> Resistor_SMD:R_0603_1608Metric
- R28: renamed from R29; footprint (none) -> Resistor_SMD:R_0603_1608Metric
- R29: renamed from R30; footprint (none) -> Resistor_SMD:R_0603_1608Metric
- R30: renamed from R27; footprint (none) -> Resistor_SMD:R_0603_1608Metric
- R31: renamed from R28; footprint (none) -> Resistor_SMD:R_0603_1608Metric
Connections:
- net GNDA: now also C35.2, C36.2, C37.2, C38.2, C39.2, C40.2, C41.2, C42.2, C43.2, C44.2, C45.2, C46.2, C47.2, C48.2, C49.2, C50.2, U14.17 (DGND), U14.2 (REF-), U14.23 (AIN2), U14.24 (AIN3), U14.6 (AVSS), Y1.2 (GND)
- net VCM: now also U14.1 (AIN4)
- net VCM_REFOUT: now also U14.4 (REFOUT)
- net at C26.1, C28.1, R30.2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: now also U14.3 (REF+)
- new net: C42.1, C43.1, U14.16 (IOVDD)
- new net: C48.3, C49.1, U14.8 (AVDD2)
- new net: C37.1, C38.1, U14.5 (REGCAPA)
- new net: U14.10 (XTAL2/CLKIO), Y1.3 (OUT)
- new net: C35.1, C36.1, U14.18 (REGCAPD)
- new net: C46.3, C47.1, U14.7 (AVDD1)
- new net: C40.1, C41.1, FB1.1, R45.2, Y1.4 (VDD)
- new net: R45.1, Y1.1 (Tri-State)
- new net +3.3V: C39.1, C42.3, C44.1, C45.1, FB1.2, R43.1, R44.1
- new net +5VA: C46.1, C48.1, C50.1
- new net AIN+: U14.21 (AIN0)
- new net AIN-: U14.22 (AIN1)
- new net DIN: U14.12 (DIN)
- new net DOUT: U14.11 (DOUT/~{RDY})
- new net SCLK: U14.13 (SCLK)
- new net ~{CS}: R43.2, U14.14 (~{CS})
- new net ~{SYNC}/~{ERR}: R44.2, U14.15 (~{SYNC}/~{ERR})
- no-connect marks 0 -> 3
Other:
- moved on the sheet: C23, C24, C25, C26, C27, C28, R27, R28, R29, R30, R31, U8A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

Commit message: Schematic
Parts:
- FB1: footprint (none) -> Inductor_SMD:L_0603_1608Metric
- R43, R44, R45: footprint (none) -> Resistor_SMD:R_0603_1608Metric
Changed lines of the file:
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@@
 	)
 	(junction
+		(at 200.66 36.83)
+		(diameter 0)
+		(color 0 0 0 0)
+	)
+	(junction
 		(at 139.7 105.41)
 		(diameter 0)
@@
 	(wire
 		(pts
+			(xy 200.66 35.56) (xy 200.66 36.83)
+		)
+		(stroke
+			(width 0)
+			(type default)
+		)
+	)
+	(wire
+		(pts
 			(xy 237.49 120.65) (xy 237.49 121.92)
 		)
@@
 		(on_board yes)
 		(dnp no)
-		(fields_autoplaced yes)
 		(property "Reference" "#PWR089"
 			(at 67.31 186.69 0)
@@
 		)
 		(property "Value" "GNDA"
-			(at 67.31 185.42 0)
+			(at 67.31 184.15 0)
 			(effects
 				(font
@@
 			)
 		)
-		(property "Footprint" ""
+		(property "Footprint" "Resistor_SMD:R_0603_1608Metric"
 			(at 187.452 80.01 90)
 			(effects
@@
 			)
 		)
-		(property "Footprint" ""
+		(property "Footprint" "Resistor_SMD:R_0603_1608Metric"
 			(at 196.342 80.01 90)
 			(effects
@@
 			)
 		)
-		(property "Footprint" ""
+		(property "Footprint" "Inductor_SMD:L_0603_1608Metric"
 			(at 255.27 38.608 90)
 			(effects
@@
 			)
 		)
-		(property "Footprint" ""
+		(property "Footprint" "Resistor_SMD:R_0603_1608Metric"
 			(at 217.17 50.038 90)
 			(effects
@@
 					(unit 1)
 				)
+			)
+		)
+	)
+	(symbol
+		(lib_id "power:PWR_FLAG")
+		(at 200.66 35.56 0)
+		(unit 1)
+		(exclude_from_sim no)
+		(in_bom yes)
+		(on_board yes)
+		(dnp no)
+		(fields_autoplaced yes)
+		(property "Reference" "#FLG04"
+			(at 200.66 33.655 0)
+			(effects
+				(font
+					(size 1.27 1.27)
+				)
+				(hide yes)
+			)
+		)
+		(property "Value" "PWR_FLAG"
+			(at 200.66 30.48 0)
+			(effects
+				(font
+					(size 1.27 1.27)
+				)
+			)
+		)
+		(property "Footprint" ""
+			(at 200.66 35.56 0)
+			(effects
+				(font
+					(size 1.27 1.27)
+				)
+				(hide yes)
+			)
+		)
+		(property "Datasheet" "~"
+			(at 200.66 35.56 0)
+			(effects
+				(font
+					(size 1.27 1.27)
+				)
+				(hide yes)
+			)
+		)
+		(property "Description" "Special symbol for telling ERC where power comes from"
+			(at 200.66 35.56 0)
+			(effects
+				(font
+					(size 1.27 1.27)
+				)
+				(hide yes)
+			)
+		)
+		(pin "1"
+		)
+		(instances
+			(project ""
+				(path "/e30159e7-fecb-4b08-a9fd-8c0b6565f013/e382cca3-340a-4115-b733-1d21769b9a67/2cbd31a6-d641-4304-8402-7aca3689c05b"
+					(reference "#FLG04")
+					(unit 1)
+				)

Commit message: Schematic and PCB
Parts:
- added C57, C58: 100n, Capacitor_SMD:C_0603_1608Metric, symbol Device:C
- C31: renamed from C50; footprint Capacitor_SMD:C_0603_1608Metric -> Capacitor_SMD:C_0805_2012Metric
- C33: renamed from C46; footprint (none) -> ADC7177M1:NFM21PC225B0J3D_MUR
- C34: renamed from C48; footprint (none) -> ADC7177M1:NFM21PC225B0J3D_MUR
- C43: renamed from C42; footprint (none) -> ADC7177M1:NFM21PC225B0J3D_MUR
- C44: footprint Capacitor_SMD:C_0603_1608Metric -> Capacitor_SMD:C_0805_2012Metric
- C45: renamed from C41; footprint Capacitor_SMD:C_0603_1608Metric -> Capacitor_SMD:C_0805_2012Metric
- renumbered C23 to C27, C25 to C28, C24 to C29, C26 to C30, C28 to C32, C27 to C35, C47 to C36, C49 to C37, C37 to C38, C38 to C39, C35 to C40, C36 to C41, C43 to C42, C45 to C46, C40 to C47, C39 to C48, R27 to R31, R30 to R32, R31 to R33, R28 to R34, R29 to R35, R43 to R36, R44 to R37, R45 to R38, U8 to U11, U9 to U12, U14 to U13
Connections:
- net +7.5V: now also C57.1, C58.1
- net GNDA: now also C57.2, C58.2

Commit message: Schematic and PCB
Parts:
- removed C33, C34, C43: NFM21PC225B0J3, ADC7177M1:NFM21PC225B0J3D_MUR, symbol Device:C_Feedthrough
- removed C42: 100n, Capacitor_SMD:C_0603_1608Metric, symbol Device:C
- removed R36, R37: 10k, Resistor_SMD:R_0603_1608Metric, symbol Device:R
- removed R38: 0, Resistor_SMD:R_0603_1608Metric, symbol Device:R
- renumbered C57 to C29, C27 to C30, C58 to C31, C28 to C32, C29 to C33, C30 to C34, C32 to C35, C31 to C36, C35 to C37, C36 to C38, C37 to C39, C38 to C40, C39 to C41, C40 to C42, C41 to C43, C46 to C45, C45 to C46, R31 to R33, R32 to R34, R33 to R35, R34 to R36, R35 to R37
Connections:
- net +3.3V: now also U13.16 (IOVDD)
- net +5VA: now also C38.1, C39.1, U13.7 (AVDD1), U13.8 (AVDD2)
- no-connect marks 3 -> 4
Other:
- moved on the sheet: C36, C38, C39, C44, C45, C46, C47, C48, FB1, Y1

Commit message: PCB
Other:
- moved on the sheet: C30, C32, C33, C34, C35, C36, C37, C38, C39, C40, C41, C42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
