File: hardware/ADC7177M1/Frontend.kicad_sch (KiCad schematic)
At the start: 61 parts, among them U1 ADG1419BRMZ, U2 ADG1419BRMZ, U3 OPA2189IDGK, U4 OPA2388IDGKx, U5 AD8066ARMZ, U6 ADG1408YRUZ, U7 ADG1408YRUZ

Commit message: Schematic
Parts:
- removed FL1: 744226, symbol Filter:Choke_CommonMode_FerriteCore_1423
- added FL1: SRF4532TA-282Y, symbol Filter:Choke_CommonMode_FerriteCore_1243
- C1, C10, C11, C12, C13, C14, C15, C16, C17, C18, C19, C2, C20, C21, C22, C3, C4, C5, C6, C7, C8, C9: footprint (none) -> Capacitor_SMD:C_0603_1608Metric
- R1, R10, R11, R12, R13, R14, R15, R16, R17, R18, R19, R2, R20, R21, R22, R23, R24, R25, R26, R3, R4, R5, R6, R7, R8, R9: footprint (none) -> Resistor_SMD:R_0603_1608Metric
- TP1: footprint (none) -> TestPoint:TestPoint_Pad_D1.5mm
- TP2, TP3: footprint (none) -> TestPoint:TestPoint_Pad_D1.5mm; now left out of the parts list
Connections:
- net at C4.1, R7.2: now also FL1.1
- net at U1.2: now also FL1.2
- net at C4.2, R8.2: now also FL1.4
- net at U2.2: now also FL1.3
Other:
- moved on the sheet: C1, C18, C19, C2, C20, C21, C22, C3, C4, R1, R10, R11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

Commit message: Schematic and PCB
Parts:
- removed FL1: SRF4532TA-282Y, symbol Filter:Choke_CommonMode_FerriteCore_1243
- removed RV1, RV2: 3269W-1-100GLF, symbol Device:R_Potentiometer_Trim
- removed TP1, TP2, TP3: TestPoint, TestPoint:TestPoint_Pad_D1.5mm, symbol Connector:TestPoint
- added L1: ACM2012-900-2P-T001, ADC7177M1:ACM2012-900-2P-T001, symbol Device:L_Ferrite_Coupled_1423
Connections:
- net at C4.1, R7.2: now also L1.1
- net at U1.2: now also L1.4
- net at C4.2, R8.2: now also L1.2
- net at U2.2: now also L1.3
- net +3V3 renamed +3.3V
Other:
- moved on the sheet: C10, C12, C14, C16, C8, R17, R18, R21, R22

Commit message: PCB
Connections:
- net REF_GND is gone; now on net GNDA: U6.9 (S8), U7.9 (S8)
Changed lines of the file:
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@@
 	(wire
 		(pts
-			(xy 119.38 63.5) (xy 130.81 63.5)
-		)
-		(stroke
-			(width 0)
-			(type default)
-		)
-	)
-	(wire
-		(pts
 			(xy 153.67 154.94) (xy 165.1 154.94)
 		)
@@
 	(wire
 		(pts
-			(xy 118.11 127) (xy 129.54 127)
-		)
-		(stroke
-			(width 0)
-			(type default)
-		)
-	)
-	(wire
-		(pts
 			(xy 119.38 181.61) (xy 119.38 180.34)
 		)
@@
 		)
 	)
-	(label "REF_GND"
-		(at 119.38 63.5 0)
-		(effects
-			(font
-				(size 1.27 1.27)
-			)
-			(justify left bottom)
-		)
-	)
-	(label "REF_GND"
-		(at 118.11 127 0)
-		(effects
-			(font
-				(size 1.27 1.27)
-			)
-			(justify left bottom)
-		)
-	)
 	(label "REF_7V"
 		(at 118.11 124.46 0)
@@
 		)
 	)
-	(hierarchical_label "REF_GND"
-		(shape input)
-		(at 118.11 127 180)
-		(effects
-			(font
-				(size 1.27 1.27)
-			)
-			(justify right)
-		)
-	)
 	(hierarchical_label "A0P"
 		(shape input)
@@
 	)
 	(symbol
+		(lib_id "power:GNDA")
+		(at 129.54 127 270)
+		(unit 1)
+		(exclude_from_sim no)
+		(in_bom yes)
+		(on_board yes)
+		(dnp no)
+		(property "Reference" "#PWR0127"
+			(at 123.19 127 0)
+			(effects
+				(font
+					(size 1.27 1.27)
+				)
+				(hide yes)
+			)
+		)
+		(property "Value" "GNDA"
+			(at 126.238 126.238 90)
+			(effects
+				(font
+					(size 1.27 1.27)
+				)
+				(justify right)
+			)
+		)
+		(property "Footprint" ""
+			(at 129.54 127 0)
+			(effects
+				(font
+					(size 1.27 1.27)
+				)
+				(hide yes)
+			)
+		)
+		(property "Datasheet" ""
+			(at 129.54 127 0)
+			(effects
+				(font
+					(size 1.27 1.27)
+				)
+				(hide yes)
+			)
+		)
+		(property "Description" "Power symbol creates a global label with name \"GNDA\" , analog ground"
+			(at 129.54 127 0)
+			(effects
+				(font
+					(size 1.27 1.27)
+				)
+				(hide yes)
+			)
+		)
+		(pin "1"
+		)
+		(instances
+			(project "ADC7177M1"
+				(path "/e30159e7-fecb-4b08-a9fd-8c0b6565f013/e382cca3-340a-4115-b733-1d21769b9a67/162a67b4-8c53-447b-9e5a-afc01ca9e483"
+					(reference "#PWR0127")
+					(unit 1)
+				)
+			)
+		)
+	)
+	(symbol
 		(lib_id "Device:R")
 		(at 237.49 30.48 90)
@@
 					(unit 1)
 				)
+			)
+		)
+	)
+	(symbol
+		(lib_id "power:GNDA")
+		(at 130.81 63.5 270)
+		(unit 1)
+		(exclude_from_sim no)
+		(in_bom yes)
+		(on_board yes)
+		(dnp no)
+		(property "Reference" "#PWR0128"
+			(at 124.46 63.5 0)
+			(effects
+				(font
+					(size 1.27 1.27)
+				)
+				(hide yes)
+			)
+		)
+		(property "Value" "GNDA"
+			(at 127.508 62.738 90)
+			(effects
+				(font
+					(size 1.27 1.27)
+				)
+				(justify right)
+			)
+		)
+		(property "Footprint" ""
+			(at 130.81 63.5 0)
+			(effects
+				(font
+					(size 1.27 1.27)
+				)
+				(hide yes)
+			)
+		)
+		(property "Datasheet" ""
+			(at 130.81 63.5 0)
+			(effects
+				(font
+					(size 1.27 1.27)
+				)
+				(hide yes)
+			)
+		)
+		(property "Description" "Power symbol creates a global label with name \"GNDA\" , analog ground"
+			(at 130.81 63.5 0)
+			(effects
+				(font
+					(size 1.27 1.27)
+				)
+				(hide yes)
+			)
+		)
+		(pin "1"
+		)
+		(instances
+			(project "ADC7177M1"
+				(path "/e30159e7-fecb-4b08-a9fd-8c0b6565f013/e382cca3-340a-4115-b733-1d21769b9a67/162a67b4-8c53-447b-9e5a-afc01ca9e483"
+					(reference "#PWR0128")
+					(unit 1)
+				)
