File: hardware/ADC7177M1/Schematic.kicad_sch (KiCad schematic)
At the start: 0 parts

Commit message: Schematic
Parts:
- added H1, H2: M3, symbol Mechanical:MountingHole
- added J1, J2: RFShield_OnePiece, symbol Device:RFShield_OnePiece
Connections:
- new net GNDA: J1.1 (Shield), J2.1 (Shield)
Other:
- added sheet IO (IO.kicad_sch)
- added sheet VREF (VREF.kicad_sch)
- sheet ADC ports: added AIN+, AIN-, DIN, DOUT, REF_5V, SCLK, VCM, ~{CS}, ~{SYNC}/~{ERR}; removed none
- sheet Frontend ports: added A0N, A0P, A1N, A1P, A2N, A2P, AIN+, AIN-, IN+, IN-, IN_CPL, REF_10V, REF_5V, REF_7V, REF_GND, VCM; removed none

Commit message: Schematic
Parts:
- H1, H2: footprint (none) -> MountingHole:MountingHole_3.2mm_M3_DIN965_Pad_TopBottom
Other:
- removed sheet IO
- added sheet Connector A (ConnectorA.kicad_sch)
- added sheet Connector B (ConnectorB.kicad_sch)

Commit message: Schematic and PCB
Parts:
- removed H1, H2: M3, MountingHole:MountingHole_3.2mm_M3_DIN965_Pad_TopBottom, symbol Mechanical:MountingHole
- J1: renamed from J2; value RFShield_OnePiece -> 3670402
- J2: renamed from J1; value RFShield_OnePiece -> 3671338
Other:
- moved on the sheet: J2
Changed lines of the file:
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@@
 	(symbol
 		(lib_id "power:GNDA")
-		(at 83.82 189.23 0)
-		(unit 1)
-		(exclude_from_sim no)
-		(in_bom yes)
-		(on_board yes)
-		(dnp no)
-		(fields_autoplaced yes)
-		(property "Reference" "#PWR01"
-			(at 83.82 195.58 0)
+		(at 76.2 189.23 0)
+		(unit 1)
+		(exclude_from_sim no)
+		(in_bom yes)
+		(on_board yes)
+		(dnp no)
+		(fields_autoplaced yes)
+		(property "Reference" "#PWR02"
+			(at 76.2 195.58 0)
 			(effects
 				(font
@@
 		)
 		(property "Value" "GNDA"
-			(at 83.82 194.31 0)
-			(effects
-				(font
-					(size 1.27 1.27)
-				)
-			)
-		)
-		(property "Footprint" ""
-			(at 83.82 189.23 0)
+			(at 76.2 194.31 0)
+			(effects
+				(font
+					(size 1.27 1.27)
+				)
+			)
+		)
+		(property "Footprint" ""
+			(at 76.2 189.23 0)
 			(effects
 				(font
@@
 		)
 		(property "Datasheet" ""
-			(at 83.82 189.23 0)
+			(at 76.2 189.23 0)
 			(effects
 				(font
@@
 		)
 		(property "Description" "Power symbol creates a global label with name \"GNDA\" , analog ground"
-			(at 83.82 189.23 0)
+			(at 76.2 189.23 0)
 			(effects
 				(font
@@
 			(project ""
 				(path "/e30159e7-fecb-4b08-a9fd-8c0b6565f013/e382cca3-340a-4115-b733-1d21769b9a67"
-					(reference "#PWR01")
-					(unit 1)
-				)
-			)
-		)
-	)
-	(symbol
-		(lib_id "Mechanical:MountingHole")
-		(at 125.73 176.53 0)
-		(unit 1)
-		(exclude_from_sim no)
-		(in_bom no)
-		(on_board yes)
-		(dnp no)
-		(fields_autoplaced yes)
-		(property "Reference" "H1"
-			(at 128.27 175.2599 0)
-			(effects
-				(font
-					(size 1.27 1.27)
-				)
-				(justify left)
-			)
-		)
-		(property "Value" "M3"
-			(at 128.27 177.7999 0)
-			(effects
-				(font
-					(size 1.27 1.27)
-				)
-				(justify left)
-			)
-		)
-		(property "Footprint" "MountingHole:MountingHole_3.2mm_M3_DIN965_Pad_TopBottom"
-			(at 125.73 176.53 0)
-			(effects
-				(font
-					(size 1.27 1.27)
-				)
-				(hide yes)
-			)
-		)
-		(property "Datasheet" "~"
-			(at 125.73 176.53 0)
-			(effects
-				(font
-					(size 1.27 1.27)
-				)
-				(hide yes)
-			)
-		)
-		(property "Description" "Mounting Hole without connection"
-			(at 125.73 176.53 0)
-			(effects
-				(font
-					(size 1.27 1.27)
-				)
-				(hide yes)
-			)
-		)
-		(instances
-			(project ""
-				(path "/e30159e7-fecb-4b08-a9fd-8c0b6565f013/e382cca3-340a-4115-b733-1d21769b9a67"
-					(reference "H1")
+					(reference "#PWR02")
 					(unit 1)
 				)
@@
 		(dnp no)
 		(fields_autoplaced yes)
-		(property "Reference" "#PWR02"
+		(property "Reference" "#PWR01"
 			(at 31.75 195.58 0)
 			(effects
@@
 			(project "ADC7177M1"
 				(path "/e30159e7-fecb-4b08-a9fd-8c0b6565f013/e382cca3-340a-4115-b733-1d21769b9a67"
-					(reference "#PWR02")
-					(unit 1)
-				)
-			)
-		)
-	)
-	(symbol
-		(lib_id "Mechanical:MountingHole")
-		(at 125.73 182.88 0)
-		(unit 1)
-		(exclude_from_sim no)
-		(in_bom no)
-		(on_board yes)
-		(dnp no)
-		(fields_autoplaced yes)
-		(property "Reference" "H2"
-			(at 128.27 181.6099 0)
-			(effects
-				(font
-					(size 1.27 1.27)
-				)
-				(justify left)
-			)
-		)
-		(property "Value" "M3"
-			(at 128.27 184.1499 0)
-			(effects
-				(font
-					(size 1.27 1.27)
-				)
-				(justify left)
-			)
-		)
-		(property "Footprint" "MountingHole:MountingHole_3.2mm_M3_DIN965_Pad_TopBottom"
-			(at 125.73 182.88 0)
-			(effects
-				(font
-					(size 1.27 1.27)
-				)
-				(hide yes)
-			)
-		)
-		(property "Datasheet" "~"
-			(at 125.73 182.88 0)
-			(effects
-				(font
-					(size 1.27 1.27)
-				)
-				(hide yes)
-			)
-		)
-		(property "Description" "Mounting Hole without connection"
-			(at 125.73 182.88 0)
-			(effects
-				(font
-					(size 1.27 1.27)
-				)
-				(hide yes)
-			)
-		)
-		(instances
-			(project "ADC7177M1"
-				(path "/e30159e7-fecb-4b08-a9fd-8c0b6565f013/e382cca3-340a-4115-b733-1d21769b9a67"
-					(reference "H2")
+					(reference "#PWR01")
 					(unit 1)
 				)
@@
 		(dnp no)
 		(fields_autoplaced yes)
-		(property "Reference" "J2"
+		(property "Reference" "J1"
 			(at 48.26 177.7999 0)
 			(effects
@@
 			)
 		)
-		(property "Value" "RFShield_OnePiece"
+		(property "Value" "3670402"
 			(at 48.26 180.3399 0)
 			(effects
@@
 			(project "ADC7177M1"
 				(path "/e30159e7-fecb-4b08-a9fd-8c0b6565f013/e382cca3-340a-4115-b733-1d21769b9a67"
+					(reference "J1")
+					(unit 1)
+				)
+			)
+		)
+	)
+	(symbol
+		(lib_id "Device:RFShield_OnePiece")
+		(at 76.2 179.07 0)
+		(unit 1)
+		(exclude_from_sim no)
+		(in_bom yes)
+		(on_board yes)
+		(dnp no)
+		(fields_autoplaced yes)
+		(property "Reference" "J2"
+			(at 92.71 177.7999 0)
+			(effects
+				(font
+					(size 1.27 1.27)
+				)
+				(justify left)
+			)
+		)
+		(property "Value" "3671338"
+			(at 92.71 180.3399 0)
+			(effects
+				(font
+					(size 1.27 1.27)
+				)
+				(justify left)
+			)
+		)
+		(property "Footprint" ""
+			(at 76.2 181.61 0)
+			(effects
+				(font
+					(size 1.27 1.27)
+				)
+				(hide yes)
+			)
+		)
+		(property "Datasheet" "~"
+			(at 76.2 181.61 0)
+			(effects
+				(font
+					(size 1.27 1.27)
+				)
+				(hide yes)
+			)
+		)
+		(property "Description" "One-piece EMI RF shielding cabinet"
+			(at 76.2 179.07 0)
+			(effects
+				(font
+					(size 1.27 1.27)
+				)
+				(hide yes)
+			)
+		)
+		(pin "1"
+		)
+		(instances
+			(project ""
+				(path "/e30159e7-fecb-4b08-a9fd-8c0b6565f013/e382cca3-340a-4115-b733-1d21769b9a67"
 					(reference "J2")
 					(unit 1)
 				)
-			)
-		)
-	)
-	(symbol
-		(lib_id "Device:RFShield_OnePiece")
-		(at 83.82 179.07 0)
-		(unit 1)
-		(exclude_from_sim no)
-		(in_bom yes)
-		(on_board yes)
-		(dnp no)
-		(fields_autoplaced yes)
-		(property "Reference" "J1"
-			(at 100.33 177.7999 0)
-			(effects
-				(font
-					(size 1.27 1.27)
-				)
-				(justify left)
-			)
-		)
-		(property "Value" "RFShield_OnePiece"
-			(at 100.33 180.3399 0)
-			(effects
-				(font
-					(size 1.27 1.27)
-				)
-				(justify left)
-			)
-		)
-		(property "Footprint" ""
-			(at 83.82 181.61 0)
-			(effects
-				(font
-					(size 1.27 1.27)
-				)
-				(hide yes)
-			)
-		)
-		(property "Datasheet" "~"
-			(at 83.82 181.61 0)
-			(effects
-				(font
-					(size 1.27 1.27)
-				)
-				(hide yes)
-			)
-		)
-		(property "Description" "One-piece EMI RF shielding cabinet"
-			(at 83.82 179.07 0)
-			(effects
-				(font
-					(size 1.27 1.27)
-				)
-				(hide yes)
-			)
-		)
-		(pin "1"
-		)
-		(instances
-			(project ""
-				(path "/e30159e7-fecb-4b08-a9fd-8c0b6565f013/e382cca3-340a-4115-b733-1d21769b9a67"
-					(reference "J1")
-					(unit 1)
-				)

Commit message: Schematic and PCB
Parts:
- J1: value 3670402 -> 3670513; footprint (none) -> ADC7177M1:3670513
- J2: value 3671338 -> 3670345; footprint (none) -> ADC7177M1:3670345
Changed lines of the file:
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@@
 			)
 		)
-		(property "Value" "3670402"
+		(property "Value" "3670513"
 			(at 48.26 180.3399 0)
 			(effects
@@
 			)
 		)
-		(property "Footprint" ""
+		(property "Footprint" "ADC7177M1:3670513"
 			(at 31.75 181.61 0)
 			(effects
@@
 			)
 		)
-		(property "Value" "3671338"
+		(property "Value" "3670345"
 			(at 92.71 180.3399 0)
 			(effects
@@
 			)
 		)
-		(property "Footprint" ""
+		(property "Footprint" "ADC7177M1:3670345"
 			(at 76.2 181.61 0)
 			(effects
@@
 		)
 		(fill
-			(color 0 0 0 0.0000)
+			(color 255 255 194 1.0000)
 		)
 		(property "Sheetname" "VREF"
@@
 		)
 		(fill
-			(color 0 0 0 0.0000)
+			(color 255 255 194 1.0000)
 		)
 		(property "Sheetname" "Frontend"
@@
 		)
 		(fill
-			(color 0 0 0 0.0000)
+			(color 255 255 194 1.0000)
 		)
 		(property "Sheetname" "Connector A"
@@
 		)
 		(fill
-			(color 0 0 0 0.0000)
+			(color 255 255 194 1.0000)
 		)
 		(property "Sheetname" "ADC"
@@
 		)
 		(fill
-			(color 0 0 0 0.0000)
+			(color 255 255 194 1.0000)
 		)
 		(property "Sheetname" "Power"
@@
 		)
 		(fill
-			(color 0 0 0 0.0000)
+			(color 255 255 194 1.0000)
 		)
 		(property "Sheetname" "Connector B"

Commit message: PCB
Parts:
- added FID1, FID2, FID3, FID4, FID5, FID6: Fiducial, Fiducial:Fiducial_0.5mm_Mask1mm, symbol Mechanical:Fiducial
Other:
- sheet Frontend ports: added none; removed REF_GND
- sheet VREF ports: added none; removed REF_GND
