File: hardware/ADC7177M1/VREF.kicad_sch (KiCad schematic)
At the start: 27 parts, among them U10 ADR1399KEZ, U11 LT1012S8, U12 ADA4522-1ARMZ, U13 AD8065ART

Commit message: Schematic
Changed lines of the file:
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@@
+	)
+	(junction
+		(at 34.29 106.68)
+		(diameter 0)
+		(color 0 0 0 0)
 	)
 	(junction
@@
 		(pts
 			(xy 218.44 109.22) (xy 219.71 109.22)
+		)
+		(stroke
+			(width 0)
+			(type default)
+		)
+	)
+	(wire
+		(pts
+			(xy 34.29 105.41) (xy 34.29 106.68)
 		)
 		(stroke
@@
 					(unit 1)
 				)
+			)
+		)
+	)
+	(symbol
+		(lib_id "power:PWR_FLAG")
+		(at 34.29 105.41 0)
+		(unit 1)
+		(exclude_from_sim no)
+		(in_bom yes)
+		(on_board yes)
+		(dnp no)
+		(fields_autoplaced yes)
+		(property "Reference" "#FLG06"
+			(at 34.29 103.505 0)
+			(effects
+				(font
+					(size 1.27 1.27)
+				)
+				(hide yes)
+			)
+		)
+		(property "Value" "PWR_FLAG"
+			(at 34.29 100.33 0)
+			(effects
+				(font
+					(size 1.27 1.27)
+				)
+			)
+		)
+		(property "Footprint" ""
+			(at 34.29 105.41 0)
+			(effects
+				(font
+					(size 1.27 1.27)
+				)
+				(hide yes)
+			)
+		)
+		(property "Datasheet" "~"
+			(at 34.29 105.41 0)
+			(effects
+				(font
+					(size 1.27 1.27)
+				)
+				(hide yes)
+			)
+		)
+		(property "Description" "Special symbol for telling ERC where power comes from"
+			(at 34.29 105.41 0)
+			(effects
+				(font
+					(size 1.27 1.27)
+				)
+				(hide yes)
+			)
+		)
+		(pin "1"
+		)
+		(instances
+			(project ""
+				(path "/e30159e7-fecb-4b08-a9fd-8c0b6565f013/e382cca3-340a-4115-b733-1d21769b9a67/0f32cb2d-c908-4fd1-b000-45b5682e819c"
+					(reference "#FLG06")
+					(unit 1)
+				)

Commit message: Schematic and PCB
Parts:
- removed TP4, TP5, TP6, TP7, TP8: TestPoint, TestPoint:TestPoint_Pad_D1.5mm, symbol Connector:TestPoint
- renumbered C29 to C49, C30 to C50, C31 to C51, C32 to C52, C33 to C53, C34 to C54, R32 to R39, R33 to R40, R34 to R41, R35 to R42, R36 to R43, R37 to R44, R38 to R45, R39 to R46, R40 to R47, R41 to R48, R42 to R49, U10 to U14, U11 to U15, U12 to U16, U13 to U17

Commit message: Schematic and PCB
Parts:
- R46: renamed from R47; now not fitted
- R47: renamed from R48; now not fitted
- renumbered R39 to R38, R40 to R39, R41 to R40, R42 to R41, R43 to R42, R44 to R43, R45 to R44, R46 to R45, R49 to R48

Commit message: PCB
Changed lines of the file:
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@@
-	)
-	(junction
-		(at 153.67 111.76)
-		(diameter 0)
-		(color 0 0 0 0)
 	)
 	(junction
@@
 	(wire
 		(pts
-			(xy 153.67 111.76) (xy 153.67 113.03)
+			(xy 153.67 110.49) (xy 153.67 113.03)
 		)
 		(stroke
@@
 	(wire
 		(pts
-			(xy 153.67 110.49) (xy 153.67 111.76)
-		)
-		(stroke
-			(width 0)
-			(type default)
-		)
-	)
-	(wire
-		(pts
 			(xy 104.14 100.33) (xy 104.14 101.6)
 		)
@@
 	(wire
 		(pts
-			(xy 160.02 111.76) (xy 153.67 111.76)
-		)
-		(stroke
-			(width 0)
-			(type default)
-		)
-	)
-	(wire
-		(pts
 			(xy 128.27 91.44) (xy 128.27 92.71)
 		)
@@
 	(wire
 		(pts
-			(xy 180.34 132.08) (xy 260.35 132.08)
-		)
-		(stroke
-			(width 0)
-			(type default)
-		)
-	)
-	(wire
-		(pts
 			(xy 33.02 177.8) (xy 45.72 177.8)
 		)
@@
 		(pts
 			(xy 34.29 105.41) (xy 34.29 106.68)
-		)
-		(stroke
-			(width 0)
-			(type default)
-		)
-	)
-	(wire
-		(pts
-			(xy 160.02 111.76) (xy 180.34 132.08)
 		)
 		(stroke
@@
 		(effects
 			(font
-				(size 1.27 1.27)
-			)
-			(justify left)
-		)
-	)
-	(hierarchical_label "REF_GND"
-		(shape output)
-		(at 260.35 132.08 0)
-		(effects
-			(font
