File: hardware/ADC7177M1/ConnectorB.kicad_sch (KiCad schematic)
At the start: 1 part, among them J4 Conn_02x08_Odd_Even

Commit message: Schematic and PCB
Parts:
- J3: renamed from J4; footprint (none) -> Connector_PinHeader_1.27mm:PinHeader_2x08_P1.27mm_Vertical_SMD
Changed lines of the file:
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@@
 		(dnp no)
 		(fields_autoplaced yes)
-		(property "Reference" "J4"
+		(property "Reference" "J3"
 			(at 127 66.04 0)
 			(effects
@@
 			)
 		)
-		(property "Footprint" ""
+		(property "Footprint" "Connector_PinHeader_1.27mm:PinHeader_2x08_P1.27mm_Vertical_SMD"
 			(at 125.73 80.01 0)
 			(effects
@@
 			(project ""
 				(path "/e30159e7-fecb-4b08-a9fd-8c0b6565f013/e382cca3-340a-4115-b733-1d21769b9a67/4e76d7a3-96d3-44e0-95f8-788ce7fa76a5"
-					(reference "J4")
+					(reference "J3")
 					(unit 1)
 				)
@@
 		(dnp no)
 		(fields_autoplaced yes)
-		(property "Reference" "#PWR099"
+		(property "Reference" "#PWR0107"
 			(at 129.54 90.17 0)
 			(effects
@@
 			(project "ADC7177M1"
 				(path "/e30159e7-fecb-4b08-a9fd-8c0b6565f013/e382cca3-340a-4115-b733-1d21769b9a67/4e76d7a3-96d3-44e0-95f8-788ce7fa76a5"
-					(reference "#PWR099")
+					(reference "#PWR0107")
 					(unit 1)
 				)
@@
 		(dnp no)
 		(fields_autoplaced yes)
-		(property "Reference" "#PWR096"
+		(property "Reference" "#PWR0105"
 			(at 124.46 90.17 0)
 			(effects
@@
 			(project ""
 				(path "/e30159e7-fecb-4b08-a9fd-8c0b6565f013/e382cca3-340a-4115-b733-1d21769b9a67/4e76d7a3-96d3-44e0-95f8-788ce7fa76a5"
-					(reference "#PWR096")
+					(reference "#PWR0105")
 					(unit 1)
 				)
@@
 		(dnp no)
 		(fields_autoplaced yes)
-		(property "Reference" "#PWR097"
+		(property "Reference" "#PWR0106"
 			(at 139.7 87.63 0)
 			(effects
@@
 			(project "ADC7177M1"
 				(path "/e30159e7-fecb-4b08-a9fd-8c0b6565f013/e382cca3-340a-4115-b733-1d21769b9a67/4e76d7a3-96d3-44e0-95f8-788ce7fa76a5"
-					(reference "#PWR097")
+					(reference "#PWR0106")
 					(unit 1)
 				)
@@
 		(dnp no)
 		(fields_autoplaced yes)
-		(property "Reference" "#PWR098"
+		(property "Reference" "#PWR0104"
 			(at 114.3 87.63 0)
 			(effects
@@
 			(project "ADC7177M1"
 				(path "/e30159e7-fecb-4b08-a9fd-8c0b6565f013/e382cca3-340a-4115-b733-1d21769b9a67/4e76d7a3-96d3-44e0-95f8-788ce7fa76a5"
-					(reference "#PWR098")
-					(unit 1)
-				)
+					(reference "#PWR0104")
+					(unit 1)
+				)

Commit message: PCB
Connections:
- net A0N: now also J3.8 (Pin_8); no longer J3.6 (Pin_6)
- net A0P: now also J3.9 (Pin_9); no longer J3.7 (Pin_7)
- net A1N: now also J3.5 (Pin_5); no longer J3.8 (Pin_8)
- net A1P: now also J3.12 (Pin_12); no longer J3.9 (Pin_9)
- net A2N: now also J3.7 (Pin_7); no longer J3.10 (Pin_10)
- net DIN: now also J3.3 (Pin_3); no longer J3.5 (Pin_5)
- net DOUT: now also J3.1 (Pin_1); no longer J3.4 (Pin_4)
- net IN_CPL: now also J3.10 (Pin_10); no longer J3.12 (Pin_12)
- net SCLK: now also J3.4 (Pin_4); no longer J3.3 (Pin_3)
- net ~{CS}: now also J3.2 (Pin_2); no longer J3.1 (Pin_1)
- net ~{SYNC}/~{ERR}: now also J3.6 (Pin_6); no longer J3.2 (Pin_2)
Changed lines of the file:
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@@
 	(hierarchical_label "A0P"
 		(shape output)
-		(at 111.76 80.01 180)
+		(at 111.76 82.55 180)
 		(effects
 			(font
@@
 	(hierarchical_label "A1P"
 		(shape output)
-		(at 111.76 82.55 180)
+		(at 142.24 85.09 0)
 		(effects
 			(font
 				(size 1.27 1.27)
 			)
-			(justify right)
+			(justify left)
 		)
 	)
 	(hierarchical_label "~{SYNC}{slash}~{ERR}"
 		(shape output)
-		(at 142.24 72.39 0)
+		(at 142.24 77.47 0)
 		(effects
 			(font
@@
 	(hierarchical_label "A1N"
 		(shape output)
-		(at 142.24 80.01 0)
+		(at 111.76 77.47 180)
+		(effects
+			(font
+				(size 1.27 1.27)
+			)
+			(justify right)
+		)
+	)
+	(hierarchical_label "~{CS}"
+		(shape output)
+		(at 142.24 72.39 0)
 		(effects
 			(font
@@
 			)
 			(justify left)
-		)
-	)
-	(hierarchical_label "~{CS}"
-		(shape output)
-		(at 111.76 72.39 180)
-		(effects
-			(font
-				(size 1.27 1.27)
-			)
-			(justify right)
 		)
 	)
@@
 	(hierarchical_label "DOUT"
 		(shape input)
+		(at 111.76 72.39 180)
+		(effects
+			(font
+				(size 1.27 1.27)
+			)
+			(justify right)
+		)
+	)
+	(hierarchical_label "A2N"
+		(shape output)
+		(at 111.76 80.01 180)
+		(effects
+			(font
+				(size 1.27 1.27)
+			)
+			(justify right)
+		)
+	)
+	(hierarchical_label "SCLK"
+		(shape output)
 		(at 142.24 74.93 0)
 		(effects
@@
 		)
 	)
-	(hierarchical_label "A2N"
+	(hierarchical_label "A0N"
 		(shape output)
-		(at 142.24 82.55 0)
+		(at 142.24 80.01 0)
 		(effects
 			(font
@@
 		)
 	)
-	(hierarchical_label "SCLK"
+	(hierarchical_label "DIN"
 		(shape output)
 		(at 111.76 74.93 180)
@@
 		)
 	)
-	(hierarchical_label "A0N"
+	(hierarchical_label "IN_CPL"
 		(shape output)
-		(at 142.24 77.47 0)
+		(at 142.24 82.55 0)
 		(effects
 			(font
-				(size 1.27 1.27)
-			)
-			(justify left)
-		)
-	)
-	(hierarchical_label "DIN"
-		(shape output)
-		(at 111.76 77.47 180)
-		(effects
-			(font
-				(size 1.27 1.27)
-			)
-			(justify right)
-		)
-	)
-	(hierarchical_label "IN_CPL"
-		(shape output)
-		(at 142.24 85.09 0)
-		(effects
-			(font

Commit message: PCB
Parts:
- J3: value Conn_02x08_Odd_Even -> FTSH-108-04-L-DV
Changed lines of the file:
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@@
 			)
 		)
-		(property "Value" "Conn_02x08_Odd_Even"
+		(property "Value" "FTSH-108-04-L-DV"
 			(at 127 68.58 0)
 			(effects
