File: hardware/ADC7177M1/ADC7177M1.kicad_pcb (KiCad board)
At the start: 2 copper layers, 132 parts, among them J3 Conn_02x08_Odd_Even, J4 Conn_02x08_Odd_Even, U1 ADG1419BRMZ, U10 ADP7182ACPZN, U11 ADA4522-2ARMZ, U12 AD8066ARMZ, U13 AD7177-2BRUZ, U14 ADR1399KEZ, U15 LT1012S8, U16 ADA4522-1ARMZ, U17 AD8065ART, U2 ADG1419BRMZ, U3 OPA2189IDGK, U4 OPA2388IDGKx, U5 AD8066ARMZ, U6 ADG1408YRUZ, U7 ADG1408YRUZ, U8 ADP7118ACPZN, U9 ADP7118ACPZN, Y1 ECS-2520MV-160-BL-TR

Commit message: Schematic and PCB
Parts:
- removed the C33 at (150.4, 64.0)
- removed the C34 at (147.6, 64.0)
- removed the C42 at (126.3, 93.1)
- removed the C43 at (116.0, 98.6)
- removed the R36 at (162.8, 73.9)
- removed the R37 at (162.8, 72.4)
- removed the R38 at (174.1, 74.2)
- added J1: 3670513, ADC7177M1:3670513, F.Cu at (149.6, 92.8)
- added J2: 3670345, ADC7177M1:3670345, B.Cu at (149.6, 92.8)
- C11, C15, C44, C54: moved to B.Cu
- C32: renamed from C28; moved to B.Cu
- C33: renamed from C29; moved to B.Cu
- C34: renamed from C30; moved to B.Cu
- C37: renamed from C35; moved to B.Cu
- C41: renamed from C39; moved to B.Cu
- C43: renamed from C41; moved to B.Cu
- C45: renamed from C46; moved to B.Cu
- C46: renamed from C45; moved to F.Cu
- C48, FB1, Y1: moved to F.Cu
- R36: renamed from R34; moved to B.Cu
- R48: renamed from R49; moved to F.Cu
- moved R30 83.1 mm to (127.8, 94.1), turned to 180 degrees
- moved R29 81.4 mm to (130.8, 94.1), turned to 180 degrees
- moved C26 74.0 mm to (130.8, 92.3), turned to 180 degrees
- moved C30 68.4 mm to (165.5, 97.8)
- moved C39 66.9 mm to (165.7, 87.1), turned to -90 degrees
- moved C33 65.8 mm to (161.7, 96.0), turned to -90 degrees
- moved R33 59.0 mm to (162.4, 97.8)
- moved C23 54.7 mm to (168.9, 99.1), turned to 180 degrees
- moved R28 52.8 mm to (167.9, 94.1), turned to 180 degrees
- moved R27 52.7 mm to (170.9, 94.1), turned to 180 degrees
- moved C36 47.8 mm to (169.0, 87.2), turned to -90 degrees
- moved C38 45.8 mm to (167.3, 87.1), turned to -90 degrees
- moved C24 45.5 mm to (171.7, 96.6), turned to -90 degrees
- moved U9 42.7 mm to (130.8, 96.3), turned to -90 degrees
- moved C44 42.5 mm to (162.1, 85.7)
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- renumbered C25 to C24, C24 to C25, C55 to C27, C56 to C28, C57 to C29, C27 to C30, C58 to C31, C32 to C35, C31 to C36, C36 to C38, C37 to C39, C38 to C40, C40 to C42, R50 to R31, R51 to R32, R31 to R33, R32 to R34, R33 to R35, R35 to R37, R39 to R38, R40 to R39, R41 to R40, R42 to R41, R43 to R42, R44 to R43, R45 to R44, R46 to R45, R47 to R46, R48 to R47
Connections:
- C38 pad 1: Net-(U13-AVDD1) -> +5VA
- C39 pad 1: Net-(U13-AVDD2) -> +5VA
- U13 pad 16: Net-(U13-IOVDD) -> +3.3V
- U13 pad 7: Net-(U13-AVDD1) -> +5VA
- U13 pad 8: Net-(U13-AVDD2) -> +5VA
- Y1 pad 1: Net-(Y1-Tri-State) -> unconnected-(Y1-Tri-State-Pad1)
Other:
- board outline added: 54 x 29 mm

Commit message: PCB
Parts:
- added FID1: Fiducial, Fiducial:Fiducial_0.5mm_Mask1mm, F.Cu at (127.4, 104.2)
- added FID2: Fiducial, Fiducial:Fiducial_0.5mm_Mask1mm, B.Cu at (127.4, 104.2)
- added FID3: Fiducial, Fiducial:Fiducial_0.5mm_Mask1mm, F.Cu at (172.6, 104.2)
- added FID4: Fiducial, Fiducial:Fiducial_0.5mm_Mask1mm, B.Cu at (127.4, 82.2)
- added FID5: Fiducial, Fiducial:Fiducial_0.5mm_Mask1mm, F.Cu at (127.4, 82.2)
- added FID6: Fiducial, Fiducial:Fiducial_0.5mm_Mask1mm, B.Cu at (172.6, 104.2)
- moved R28 9.21 mm to (170.3, 103.0), turned to 0 degrees
- moved R27 7.12 mm to (168.3, 100.7), turned to -90 degrees
- moved C23 4.55 mm to (172.8, 101.3), turned to -90 degrees
- moved U8 4.31 mm to (170.4, 100.8), turned to 0 degrees
- moved C25 3.42 mm to (130.0, 98.7), turned to 180 degrees
- moved C24 2.85 mm to (169.3, 98.2), turned to 0 degrees
- moved C4 2.59 mm to (135.1, 87.8)
- moved R30 1.85 mm to (128.3, 95.9), turned to -90 degrees
- moved C16 1.78 mm to (141.9, 93.6)
- moved C27 1.42 mm to (129.2, 86.7)
- moved R26 1.02 mm to (152.1, 86.2)
- moved C13 1.02 mm to (141.9, 89.5)
- moved C36 1.02 mm to (170.1, 87.2)
- moved U10 0.81 mm to (131.4, 86.1)
- moved C38 0.64 mm to (167.9, 87.1)
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Connections:
- J3 pad 1: /Schematic/ADC/~{CS} -> /Schematic/ADC/DOUT
- J3 pad 10: /Schematic/Connector B/A2N -> /Schematic/Frontend/IN_CPL
- J3 pad 12: /Schematic/Frontend/IN_CPL -> /Schematic/Connector B/A1P
- J3 pad 2: /Schematic/ADC/~{SYNC}/~{ERR} -> /Schematic/ADC/~{CS}
- J3 pad 3: /Schematic/ADC/SCLK -> /Schematic/ADC/DIN
- J3 pad 4: /Schematic/ADC/DOUT -> /Schematic/ADC/SCLK
- J3 pad 5: /Schematic/ADC/DIN -> /Schematic/Connector B/A1N
- J3 pad 6: /Schematic/Connector B/A0N -> /Schematic/ADC/~{SYNC}/~{ERR}
- J3 pad 7: /Schematic/Connector B/A0P -> /Schematic/Connector B/A2N
- J3 pad 8: /Schematic/Connector B/A1N -> /Schematic/Connector B/A0N
- J3 pad 9: /Schematic/Connector B/A1P -> /Schematic/Connector B/A0P
Routing:
- net +15V: track 0.00 -> 132.0 mm, vias 0 -> 14
- net +3.3V: track 0.00 -> 96.1 mm, vias 0 -> 8
- net +7.5V: track 0.00 -> 87.0 mm, vias 0 -> 5
- net -15V: track 0.00 -> 86.8 mm, vias 0 -> 7
- net +5VA: track 0.00 -> 65.0 mm, vias 0 -> 5
- net /Schematic/Frontend/IN_CPL: track 0.00 -> 62.3 mm, vias 0 -> 3
- net /Schematic/ADC/VCM: track 0.00 -> 61.5 mm, vias 0 -> 5
- net /Schematic/REF_5V: track 0.00 -> 59.4 mm, vias 0 -> 5
- net /Schematic/Frontend/REF_7V: track 0.00 -> 44.5 mm, vias 0 -> 4
- net /Schematic/Connector B/A0N: track 0.00 -> 42.2 mm, vias 0 -> 2
- net /Schematic/Connector B/A2N: track 0.00 -> 38.8 mm, vias 0 -> 2
- net /Schematic/Connector B/A1N: track 0.00 -> 38.0 mm, vias 0 -> 2
- net -2V5: track 0.00 -> 35.0 mm, vias 0 -> 3
- net /Schematic/Connector B/A2P: track 0.00 -> 34.7 mm, vias 0 -> 2
- net /Schematic/Connector B/A1P: track 0.00 -> 33.5 mm, vias 0 -> 2
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- added copper zone on F.Cu, net +15V
- added copper zone on In2.Cu, net +15V
- added copper zone on F.Cu, net +3.3V
- added copper zone on F.Cu, net +5VA
- added copper zone on In3.Cu, net +5VA
- added copper zone on F.Cu, net +5VD
- added copper zone on F.Cu, net +7.5V
- added copper zone on In3.Cu, net +7.5V
- added copper zone on F.Cu, net -15V
- added copper zone on In2.Cu, net -15V
- added copper zone on F.Cu, net -2V5
- added copper zone on In3.Cu, net -2V5
- added copper zone on B.Cu, net GNDA
- added copper zone on F.Cu, net GNDA
- added copper zone on In1.Cu, net GNDA
- added copper zone on In4.Cu, net GNDA
Other:
- outline, holes or cut-outs redrawn
- copper layers 2 -> 6
- board text added: "1"
- board text added: "2"
- board text added: "3"
- board text added: "4"
- board text added: "5"
- board text added: "6"
- board text added: "ADC7177M1 V1.0"

Commit message: PCB and schematic
Parts:
- moved J3 0.50 mm to (172.0, 95.5)
- moved C23 0.25 mm to (172.8, 101.6)
Routing:
- net /Schematic/ADC/VCM: track 61.5 -> 59.5 mm, vias 5 -> 6
- net GNDA: track 32.6 -> 33.9 mm, vias 116 -> 131
- net +15V: track 132.0 -> 130.9 mm
- net /Schematic/Frontend/REF_7V: track 44.5 -> 43.8 mm
- net /Schematic/ADC/~{SYNC}/~{ERR}: track 20.5 -> 21.1 mm
- net /Schematic/Frontend/IN_CPL: track 62.3 -> 62.8 mm
- net /Schematic/Connector B/A2N: track 38.8 -> 39.3 mm
- net /Schematic/Connector B/A0N: track 42.2 -> 42.7 mm
- net /Schematic/Connector B/A1N: track 38.0 -> 38.5 mm
- net +3.3V: track 96.1 -> 96.3 mm, vias 8 -> 9
- added copper zone on B.Cu, net +3.3V
- added copper zone on In2.Cu, net +3.3V
- added copper zone on In3.Cu, net +3.3V
- added copper zone on In2.Cu, net GNDA
- added copper zone on In3.Cu, net GNDA

Commit message: PCB
Parts:
- moved C26 7.24 mm to (130.7, 99.6), turned to 0 degrees
- moved C25 5.64 mm to (131.4, 93.2), turned to 0 degrees
- moved R30 4.95 mm to (133.2, 96.0), turned to 90 degrees
- moved R29 3.70 mm to (130.9, 97.8), turned to 0 degrees
- moved J4 3.50 mm to (127.0, 93.0)
- moved FID1 3.48 mm to (126.1, 101.0)
- moved FID2 3.48 mm to (126.1, 101.0)
- moved J3 2.50 mm to (172.0, 93.0)
- moved U9 0.74 mm to (130.9, 95.6), turned to 90 degrees
Routing:
- net -15V: track 86.5 -> 27.7 mm, vias 7 -> 8
- net +7.5V: track 86.6 -> 68.4 mm, vias 5 -> 6
- net +5VA: track 65.0 -> 69.5 mm
- net /Schematic/Frontend/IN_CPL: track 62.8 -> 60.2 mm
- net /Schematic/ADC/~{SYNC}/~{ERR}: track 21.1 -> 18.6 mm
- net /Schematic/Connector B/A2N: track 39.3 -> 36.8 mm
- net /Schematic/Connector B/A1N: track 38.5 -> 36.0 mm
- net /Schematic/Connector B/A0N: track 42.7 -> 40.2 mm
- net /Schematic/ADC/~{CS}: track 19.5 -> 17.4 mm
- net /Schematic/Connector A/IN+: track 21.1 -> 23.1 mm
- net /Schematic/ADC/SCLK: track 21.7 -> 19.9 mm
- net /Schematic/ADC/DIN: track 20.0 -> 18.3 mm
- net Net-(U6-S2): track 9.31 -> 7.64 mm, vias 1 -> 0
- net /Schematic/ADC/DOUT: track 17.3 -> 15.8 mm
- net +15V: track 130.9 -> 129.9 mm, vias 14 -> 12
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
Commit message: PCB
Parts:
- J3, J4: value Conn_02x08_Odd_Even -> FTSH-108-04-L-DV
Routing:
- net GNDA: vias 125 -> 105
