File: hardware/ADC7177B1/Ethernet.kicad_sch (KiCad schematic)
At the start: 25 parts, among them J2 RJ45_Wuerth_7499010121A, U3 LAN8742A, Y2 NX5032GA-25

Commit message: PCB
Parts:
- Y2: footprint ETH1HMSR-SMS:NX5032GA -> ADC7177B1:NX5032GA
Changed lines of the file:
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@@
 			)
 		)
-		(property "Description" ""
+		(property "Description" "4 resistor network, parallel topology"
 			(at 175.26 40.64 0)
 			(effects
@@
 			)
 		)
-		(property "Description" ""
+		(property "Description" "4 resistor network, parallel topology"
 			(at 72.39 88.9 0)
 			(effects
@@
 			)
 		)
-		(property "Description" ""
+		(property "Description" "LAN8720 Ethernet PHY with RMII interface, QFN-24"
 			(at 113.03 91.44 0)
 			(effects
@@
 			)
 		)
-		(property "Description" ""
+		(property "Description" "4 resistor network, parallel topology"
 			(at 96.52 168.91 0)
 			(effects
@@
 			)
 		)
-		(property "Footprint" "ETH1HMSR-SMS:NX5032GA"
+		(property "Footprint" "ADC7177B1:NX5032GA"
 			(at 80.01 125.73 0)
 			(effects

Commit message: PCB
Parts:
- renumbered C15 to C16, C16 to C17, C17 to C18, C18 to C19, C19 to C20, C20 to C21, C21 to C22, C22 to C23, C23 to C24, C24 to C25, C25 to C26, C26 to C27
Changed lines of the file:
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@@
 		(on_board yes)
 		(dnp no)
-		(property "Reference" "C18"
+		(property "Reference" "C19"
 			(at 93.091 129.6416 0)
 			(effects
@@
 			(project "ETH1HMSR-SMS"
 				(path "/06a56fb9-779c-428e-b281-14ac9294755f/ce8ead21-c650-4940-b61e-074f59a08930/21ee60a8-817f-4081-bcd1-9c2a5024e4a1"
-					(reference "C18")
+					(reference "C19")
 					(unit 1)
 				)
@@
 		(on_board yes)
 		(dnp no)
-		(property "Reference" "C22"
+		(property "Reference" "C23"
 			(at 133.731 35.6616 0)
 			(effects
@@
 			(project "ETH1HMSR-SMS"
 				(path "/06a56fb9-779c-428e-b281-14ac9294755f/ce8ead21-c650-4940-b61e-074f59a08930/21ee60a8-817f-4081-bcd1-9c2a5024e4a1"
-					(reference "C22")
+					(reference "C23")
 					(unit 1)
 				)
@@
 		(on_board yes)
 		(dnp no)
-		(property "Reference" "C21"
+		(property "Reference" "C22"
 			(at 122.301 35.6616 0)
 			(effects
@@
 			(project "ETH1HMSR-SMS"
 				(path "/06a56fb9-779c-428e-b281-14ac9294755f/ce8ead21-c650-4940-b61e-074f59a08930/21ee60a8-817f-4081-bcd1-9c2a5024e4a1"
-					(reference "C21")
+					(reference "C22")
 					(unit 1)
 				)
@@
 		(on_board yes)
 		(dnp no)
-		(property "Reference" "C17"
+		(property "Reference" "C18"
 			(at 82.931 53.4416 0)
 			(effects
@@
 			(project "ETH1HMSR-SMS"
 				(path "/06a56fb9-779c-428e-b281-14ac9294755f/ce8ead21-c650-4940-b61e-074f59a08930/21ee60a8-817f-4081-bcd1-9c2a5024e4a1"
-					(reference "C17")
+					(reference "C18")
 					(unit 1)
 				)
@@
 		(on_board yes)
 		(dnp no)
-		(property "Reference" "C15"
+		(property "Reference" "C16"
 			(at 71.501 129.6416 0)
 			(effects
@@
 			(project "ETH1HMSR-SMS"
 				(path "/06a56fb9-779c-428e-b281-14ac9294755f/ce8ead21-c650-4940-b61e-074f59a08930/21ee60a8-817f-4081-bcd1-9c2a5024e4a1"
-					(reference "C15")
+					(reference "C16")
 					(unit 1)
 				)
@@
 		(on_board yes)
 		(dnp no)
-		(property "Reference" "C26"
+		(property "Reference" "C27"
 			(at 213.741 101.7016 0)
 			(effects
@@
 			(project "ETH1HMSR-SMS"
 				(path "/06a56fb9-779c-428e-b281-14ac9294755f/ce8ead21-c650-4940-b61e-074f59a08930/21ee60a8-817f-4081-bcd1-9c2a5024e4a1"
-					(reference "C26")
+					(reference "C27")
 					(unit 1)
 				)
@@
 		(on_board yes)
 		(dnp no)
-		(property "Reference" "C23"
+		(property "Reference" "C24"
 			(at 145.161 35.6616 0)
 			(effects
@@
 			(project "ETH1HMSR-SMS"
 				(path "/06a56fb9-779c-428e-b281-14ac9294755f/ce8ead21-c650-4940-b61e-074f59a08930/21ee60a8-817f-4081-bcd1-9c2a5024e4a1"
-					(reference "C23")
+					(reference "C24")
 					(unit 1)
 				)
@@
 		(on_board yes)
 		(dnp no)
-		(property "Reference" "C16"
+		(property "Reference" "C17"
 			(at 82.931 35.6616 0)
 			(effects
@@
 			(project "ETH1HMSR-SMS"
 				(path "/06a56fb9-779c-428e-b281-14ac9294755f/ce8ead21-c650-4940-b61e-074f59a08930/21ee60a8-817f-4081-bcd1-9c2a5024e4a1"
-					(reference "C16")
+					(reference "C17")
 					(unit 1)
 				)
@@
 		(on_board yes)
 		(dnp no)
-		(property "Reference" "C19"
+		(property "Reference" "C20"
 			(at 94.361 35.6616 0)
 			(effects
@@
 			(project "ETH1HMSR-SMS"
 				(path "/06a56fb9-779c-428e-b281-14ac9294755f/ce8ead21-c650-4940-b61e-074f59a08930/21ee60a8-817f-4081-bcd1-9c2a5024e4a1"
-					(reference "C19")
+					(reference "C20")
 					(unit 1)
 				)
@@
 		(on_board yes)
 		(dnp no)
-		(property "Reference" "C25"
+		(property "Reference" "C26"
 			(at 202.311 35.6616 0)
 			(effects
@@
 			(project "ETH1HMSR-SMS"
 				(path "/06a56fb9-779c-428e-b281-14ac9294755f/ce8ead21-c650-4940-b61e-074f59a08930/21ee60a8-817f-4081-bcd1-9c2a5024e4a1"
-					(reference "C25")
+					(reference "C26")
 					(unit 1)
 				)
@@
 		(on_board yes)
 		(dnp no)
-		(property "Reference" "C20"
+		(property "Reference" "C21"
 			(at 94.361 53.4416 0)
 			(effects
@@
 			(project "ETH1HMSR-SMS"
 				(path "/06a56fb9-779c-428e-b281-14ac9294755f/ce8ead21-c650-4940-b61e-074f59a08930/21ee60a8-817f-4081-bcd1-9c2a5024e4a1"
-					(reference "C20")
+					(reference "C21")
 					(unit 1)
 				)
@@
 		(on_board yes)
 		(dnp no)
-		(property "Reference" "C24"
+		(property "Reference" "C25"
 			(at 160.401 35.6616 0)
 			(effects
@@
 			(project "ETH1HMSR-SMS"
 				(path "/06a56fb9-779c-428e-b281-14ac9294755f/ce8ead21-c650-4940-b61e-074f59a08930/21ee60a8-817f-4081-bcd1-9c2a5024e4a1"
-					(reference "C24")
+					(reference "C25")
 					(unit 1)
 				)
