File: hardware/ADC7177B1/Frontend.kicad_sch (KiCad schematic)
At the start: 29 parts, among them J3 Conn_01x01, J4 Conn_01x01, K1 SILxx-1Axx-71x, K2 SILxx-1Axx-71x, U8 AD8599ARZ

Commit message: Schematic
Parts:
- removed K1, K2: SILxx-1Axx-71x, Relay_THT:Relay_SPST_StandexMeder_SIL_Form1A, symbol Relay:SILxx-1Axx-71x
- added D4, D5: 1N4148W, Diode_SMD:D_SOD-123, symbol Diode:1N4148W
- added K1: G6SK-2F-DC5, symbol Relay:G6SK-2
- added Q3, Q4: MMBT3904, Package_TO_SOT_SMD:SOT-23, symbol Transistor_BJT:MMBT3904
- added R34, R41: 1k2, Resistor_SMD:R_0603_1608Metric_Pad0.98x0.95mm_HandSolder, symbol Device:R
- added R44, R45: 10k, symbol Device:R
- added U10, U9: CPC1002N, Package_SO:SOP-4_3.8x4.1mm_P2.54mm, symbol Relay_SolidState:CPC1002N
- R20, R31: footprint (none) -> Resistor_SMD:R_1206_3216Metric_Pad1.30x1.75mm_HandSolder
- R21: renamed from R26; footprint (none) -> Resistor_SMD:R_1206_3216Metric_Pad1.30x1.75mm_HandSolder
- R22: renamed from R21; footprint (none) -> Resistor_SMD:R_1206_3216Metric_Pad1.30x1.75mm_HandSolder
- R23: renamed from R27; footprint (none) -> Resistor_SMD:R_1206_3216Metric_Pad1.30x1.75mm_HandSolder
- R24: renamed from R22; footprint (none) -> Resistor_SMD:R_1206_3216Metric_Pad1.30x1.75mm_HandSolder
- R25: renamed from R28; footprint (none) -> Resistor_SMD:R_1206_3216Metric_Pad1.30x1.75mm_HandSolder
- R26: renamed from R23; footprint (none) -> Resistor_SMD:R_1206_3216Metric_Pad1.30x1.75mm_HandSolder
- R27: renamed from R29; footprint (none) -> Resistor_SMD:R_1206_3216Metric_Pad1.30x1.75mm_HandSolder
- R28: renamed from R25; footprint (none) -> Resistor_SMD:R_1206_3216Metric_Pad1.30x1.75mm_HandSolder
- R29: renamed from R30; footprint (none) -> Resistor_SMD:R_1206_3216Metric_Pad1.30x1.75mm_HandSolder
- R30: renamed from R24; footprint (none) -> Resistor_SMD:R_1206_3216Metric_Pad1.30x1.75mm_HandSolder
- R32, R33: footprint (none) -> Resistor_SMD:R_0603_1608Metric_Pad0.98x0.95mm_HandSolder
- R35: renamed from R36; value 1k/0.1% -> 10k/0.1%; footprint (none) -> Resistor_SMD:R_0603_1608Metric_Pad0.98x0.95mm_HandSolder
- R36: renamed from R38; value 1k5 -> DNP; footprint (none) -> Resistor_SMD:R_0603_1608Metric_Pad0.98x0.95mm_HandSolder; now not fitted; now left out of the parts list
- R37: renamed from R34; value 1k/0.1% -> 10k/0.1%; footprint (none) -> Resistor_SMD:R_0603_1608Metric_Pad0.98x0.95mm_HandSolder
- R38: renamed from R39; value 120/0.05% -> 1100/0.1%; footprint (none) -> Resistor_SMD:R_0603_1608Metric_Pad0.98x0.95mm_HandSolder
- R39: renamed from R37; value 1k/0.1% -> 10k/0.1%; footprint (none) -> Resistor_SMD:R_0603_1608Metric_Pad0.98x0.95mm_HandSolder; now not fitted; now left out of the parts list
- R40: renamed from R35; value 1k/0.1% -> 10k/0.1%; footprint (none) -> Resistor_SMD:R_0603_1608Metric_Pad0.98x0.95mm_HandSolder; now not fitted; now left out of the parts list
- R42: renamed from R40; value 1k -> 1k2; footprint (none) -> Resistor_SMD:R_0603_1608Metric_Pad0.98x0.95mm_HandSolder
- R43: renamed from R41; value 10.2/0.05% -> 110/0.05%; footprint (none) -> Resistor_SMD:R_0603_1608Metric_Pad0.98x0.95mm_HandSolder
Connections:
- net +5VD: now also D4.1 (K), D5.1 (K), K1.1, K1.6
- net GND: now also Q3.2 (E), Q4.2 (E), U10.2, U9.2
- net at R37.1, R40.1, U8.6 (-): now also U10.3, U9.3
- net at R37.2, R40.2, U8.7: now also K1.3
- net at R42.2, R43.2: now also U10.4
- net at R35.2, R39.2, U8.1: now also K1.10
- net at R36.2, R38.2: now also U9.4
- new net: R34.2, U9.1
- new net: R41.2, U10.1
- new net: D5.2 (A), K1.7, Q4.3 (C)
- new net: Q3.1 (B), R44.2
- new net: D4.2 (A), K1.12, Q3.3 (C)
- new net: Q4.1 (B), R45.2
- new net IN+: K1.9
- new net IN-: K1.4
- new net MCU_Gx10: R34.1
- new net MCU_Gx100: R41.1
Other:
- moved on the sheet: J3, J4, R20, R21, R22, R23, R24, R25, R26, R27, R28, R29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

Commit message: PCB
Parts:
- added C58, C59, C60, C61, C62, C63, C64, C65: 0.1u, Capacitor_SMD:C_0603_1608Metric_Pad1.08x0.95mm_HandSolder, symbol Device:C
- added J6, J7: Conn_01x01, ADC7177B1:S16N-PC, symbol Connector_Generic:Conn_01x01
- added R50, R51, R56, R58, R61, R62: 510, Resistor_SMD:R_0603_1608Metric_Pad0.98x0.95mm_HandSolder, symbol Device:R
- added U13: AD8599ARZ, Package_SO:SOIC-8_3.9x4.9mm_P1.27mm, symbol ADC7177B1:AD8599ARZ
- J4: renamed from J3; footprint (none) -> ADC7177B1:S16N-PC
- J5: renamed from J4; footprint (none) -> ADC7177B1:S16N-PC
- K1: footprint (none) -> ADC7177B1:G6SK-2F
- R59: renamed from R45; footprint (none) -> Resistor_SMD:R_0603_1608Metric_Pad0.98x0.95mm_HandSolder
- R60: renamed from R44; footprint (none) -> Resistor_SMD:R_0603_1608Metric_Pad0.98x0.95mm_HandSolder
- renumbered D5 to D7, D4 to D8, Q4 to Q6, Q3 to Q7, R20 to R31, R21 to R32, R22 to R33, R23 to R34, R24 to R35, R25 to R36, R26 to R37, R27 to R38, R28 to R39, R29 to R40, R30 to R41, R31 to R42, R32 to R43, R33 to R44, R34 to R45, R35 to R46, R36 to R47, R37 to R48, R38 to R49, R39 to R52, R40 to R53, R41 to R54, R42 to R55, R43 to R57, U8 to U12, U9 to U14, U10 to U15
Connections:
- net +15V: now also C58.1, C60.1, U13.8 (V+)
- net -15V: now also C59.1, C61.1, U13.4 (V-)
- net GND: now also C58.2, C59.2, C60.2, C61.2, C62.2, C63.1, C64.1, C65.1
- net at R44.2, U12.5 (+): now also C64.2
- net at R48.2, R53.2, U12.7: now also R58.1; no longer K1.3
- net at R46.2, R52.2, U12.1: now also R56.1; no longer K1.10
- net at R43.2, U12.3 (+): now also C65.2
- net RLY_S: now reaches R60.1
- net at K1.5: now also R51.2
- net at K1.8: now also R50.2
- net RLY_R: now reaches R59.1
- net MCU_Gx10 renamed Gx10
- net MCU_Gx100 renamed Gx100
- new net: J7.1 (Pin_1), R62.1
- new net: J6.1 (Pin_1), R61.1
- new net: C62.1, R61.2, U13.3 (+)
- new net: K1.10, R56.2
- new net: C63.2, R62.2, U13.5 (+)
- new net: R51.1, U13.6 (-), U13.7
- new net: K1.3, R58.2
- new net: R50.1, U13.1, U13.2 (-)
Other:
- moved on the sheet: D7, D8, J4, J5, K1, Q6, Q7, R31, R32, R33, R34, R35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

Commit message: PCB
Parts:
- R51: renamed from R49; value 1100/0.1% -> 1k1/0.1%
- renumbered C58 to C60, C59 to C61, C60 to C62, C61 to C63, C65 to C64, C64 to C65, C62 to C66, C63 to C67, R61 to R45, R62 to R46, R45 to R47, R46 to R48, R47 to R49, R48 to R50, R50 to R52, R51 to R53, R52 to R54, R53 to R55, R54 to R56, R55 to R57, R56 to R58, R57 to R59, R58 to R60, R59 to R61, R60 to R62
