File: hardware/ADC7177B1/Power.kicad_sch (KiCad schematic)
At the start: 33 parts, among them Q2 FZT851, Q3 FZT951, U4 THN 15-2425, U5 TPS7A4901DGN, U7 TPS7A3001DGN

Commit message: Schematic
Parts:
- C37: renamed from C38; footprint (none) -> Capacitor_SMD:C_0603_1608Metric_Pad1.08x0.95mm_HandSolder
- C38: renamed from C40; footprint (none) -> Capacitor_SMD:C_0603_1608Metric_Pad1.08x0.95mm_HandSolder
- C39: renamed from C37; footprint (none) -> Capacitor_SMD:C_0603_1608Metric_Pad1.08x0.95mm_HandSolder
- C40: renamed from C41; footprint (none) -> Capacitor_SMD:C_0603_1608Metric_Pad1.08x0.95mm_HandSolder
- R12: renamed from R13; footprint (none) -> Resistor_SMD:R_0603_1608Metric_Pad0.98x0.95mm_HandSolder
- R13: renamed from R14; footprint (none) -> Resistor_SMD:R_0603_1608Metric_Pad0.98x0.95mm_HandSolder
- R14: renamed from R12; footprint (none) -> Resistor_SMD:R_0603_1608Metric_Pad0.98x0.95mm_HandSolder
- R15, R16, R17, R18, R19: footprint (none) -> Resistor_SMD:R_0603_1608Metric_Pad0.98x0.95mm_HandSolder
- renumbered C30 to C27, C32 to C28, C33 to C30, C28 to C31, C34 to C32, C27 to C33, C35 to C34, C31 to C35, C39 to C41, Q2 to Q1, Q3 to Q2, U7 to U6

Commit message: PCB
Parts:
- added C29, C32, C35, C38, C41, C52, C53, C54, C57: 10u/50V, Capacitor_SMD:C_1206_3216Metric_Pad1.33x1.80mm_HandSolder, symbol Device:C
- added C44, C45, C48, C49, C55, C56: 10n, Capacitor_SMD:C_0603_1608Metric_Pad1.08x0.95mm_HandSolder, symbol Device:C
- added D2: BZX84C10LT1G, Package_TO_SOT_SMD:SOT-23, symbol Diode:BZX84Cxx
- added D3: 1N4148W, Diode_SMD:D_SOD-123, symbol Diode:1N4148W
- added D6: SS16, Diode_SMD:D_SMA, symbol Diode:SS16
- added J3: 1715721, TerminalBlock_Phoenix:TerminalBlock_Phoenix_MKDS-1,5-2_1x02_P5.00mm_Horizontal, symbol Connector_Generic:Conn_01x02
- added L3: 10u, symbol Device:L
- added Q1: SI5618A, Package_TO_SOT_SMD:SOT-23, symbol Device:Q_PMOS_GSD
- added Q2: MMBT3904, Package_TO_SOT_SMD:SOT-23, symbol Transistor_BJT:MMBT3904
- added Q5: FZT851, Package_TO_SOT_SMD:SOT-223, symbol Transistor_BJT:Q_NPN_BCEC
- added R12: 0, Resistor_SMD:R_1206_3216Metric_Pad1.30x1.75mm_HandSolder, symbol Device:R
- added R13, R14: 100k, Resistor_SMD:R_0603_1608Metric_Pad0.98x0.95mm_HandSolder, symbol Device:R
- added R17, R20: 1k, Resistor_SMD:R_0603_1608Metric_Pad0.98x0.95mm_HandSolder, symbol Device:R
- added R25, R27, R29: 120k, Resistor_SMD:R_0603_1608Metric_Pad0.98x0.95mm_HandSolder, symbol Device:R
- added R26, R28, R30: 10k, Resistor_SMD:R_0603_1608Metric_Pad0.98x0.95mm_HandSolder, symbol Device:R
- added U10, U8, U9: TPS7A4901DGN, Package_SO:HVSSOP-8-1EP_3x3mm_P0.65mm_EP1.57x1.89mm_ThermalVias, symbol ADC7177B1:TPS7A4901DGN
- added U5: TEC 3-2419WI, Converter_DCDC:Converter_DCDC_TRACO_TEC3-24xxUI_THT, symbol Converter_DCDC:TEC3-2411UI
- C27, C28: footprint (none) -> Capacitor_SMD:C_1206_3216Metric_Pad1.33x1.80mm_HandSolder
- C30: renamed from C29; footprint (none) -> Capacitor_SMD:C_1206_3216Metric_Pad1.33x1.80mm_HandSolder
- C31: renamed from C30; footprint (none) -> Capacitor_SMD:C_1206_3216Metric_Pad1.33x1.80mm_HandSolder
- C33: renamed from C31; footprint (none) -> Capacitor_SMD:C_1206_3216Metric_Pad1.33x1.80mm_HandSolder
- C34: renamed from C32; footprint (none) -> Capacitor_SMD:C_1206_3216Metric_Pad1.33x1.80mm_HandSolder
- C36: renamed from C33; footprint (none) -> Capacitor_SMD:C_1206_3216Metric_Pad1.33x1.80mm_HandSolder
- C37: renamed from C34; footprint (none) -> Capacitor_SMD:C_1206_3216Metric_Pad1.33x1.80mm_HandSolder
- C39: renamed from C35; footprint (none) -> Capacitor_SMD:C_1206_3216Metric_Pad1.33x1.80mm_HandSolder
- C40: renamed from C36; footprint (none) -> Capacitor_SMD:C_1206_3216Metric_Pad1.33x1.80mm_HandSolder
- C50: renamed from C41; value 10u/35V -> 10u/50V; footprint (none) -> Capacitor_SMD:C_1206_3216Metric_Pad1.33x1.80mm_HandSolder
- C51: renamed from C42; value 10u/35V -> 10u/50V; footprint (none) -> Capacitor_SMD:C_1206_3216Metric_Pad1.33x1.80mm_HandSolder
- Q3: renamed from Q1; footprint (none) -> Package_TO_SOT_SMD:SOT-223
- Q4: renamed from Q2; footprint (none) -> Package_TO_SOT_SMD:SOT-223
- U4: footprint (none) -> ADC7177B1:THN_15-2425; symbol ADC7177B1:TBA1-0521E -> ADC7177B1:THN 15-2425
- renumbered C37 to C42, C38 to C43, C39 to C46, C40 to C47, D2 to D4, D3 to D5, R12 to R15, R13 to R16, R14 to R18, R15 to R19, R16 to R21, R17 to R22, R18 to R23, R19 to R24, U5 to U6, U6 to U7
Connections:
- net +24V: now also D2.3 (K), D3.2 (A), Q1.2 (S), Q2.2 (E), R12.2, U5.2 (+Vin)
- net GND: now also U4.4 (Com), C29.2, C32.2, C35.2, C38.2, C41.2, C44.2, C45.2, C52.2, C53.2, C54.2, C55.2, C57.2, R26.2, R28.2, R30.2, U10.4 (GND), U10.9 (EP), U5.7 (-Vout), U8.4 (GND), U8.9 (EP), U9.4 (GND), U9.9 (EP); no longer U4.3 (Com)
- net GNDS: now also J3.2 (Pin_2), R13.2, R14.2, U5.1 (-Vin)
- new net: C35.1, R17.1, R20.1
- new net: C32.1, D6.1 (K), L3.2, Q5.2 (C), Q5.4 (C), R17.2
- new net: C29.1, L3.1, U5.6 (+Vout)
- new net: C56.2, R29.2, R30.1, U10.2 (FB)
- new net: C55.1, U10.6 (NR/SS)
- new net: D2.1 (A), Q1.1 (G), Q2.3 (C), R13.1
- new net: J3.1 (Pin_1), Q1.3 (D), R12.1
- new net: C48.2, R25.2, R26.1, U8.2 (FB)
- new net: C41.1, D6.2 (A), Q5.3 (E), U8.5 (EN), U8.8 (IN), U9.5 (EN), U9.8 (IN)
- new net: C49.2, R27.2, R28.1, U9.2 (FB)
- new net: D3.1 (K), Q2.1 (B), R14.1
- new net: C38.1, Q5.1 (B), R20.2
- new net: C45.1, U9.6 (NR/SS)
- new net: C44.1, U8.6 (NR/SS)
- new net +3.3V: C56.1, C57.1, R29.1, U10.1 (OUT)
- new net +5VA: C48.1, C52.1, R25.1, U8.1 (OUT)
- new net +5VD: C49.1, C53.1, C54.1, R27.1, U10.5 (EN), U10.8 (IN), U9.1 (OUT)
- no-connect marks 1 -> 2
Other:
- note added: "Reverse voltage protection"
- moved on the sheet: C27, C28, C30, C31, C33, C34, C36, C37, C39, C40, C42, C43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

Commit message: PCB
Parts:
- added C43: 10u/50V, Capacitor_SMD:C_1206_3216Metric_Pad1.33x1.80mm_HandSolder, symbol Device:C
- L1, L2, L3: value 10u -> 74408943100; footprint (none) -> ADC7177B1:74408943100
- renumbered C27 to C28, C28 to C29, C29 to C30, C30 to C31, C31 to C32, C32 to C33, C33 to C34, C34 to C35, C35 to C36, C36 to C37, C37 to C38, C38 to C39, C39 to C40, C40 to C41, C41 to C42, C42 to C44, C43 to C45, C44 to C46, C45 to C47, C46 to C48, C47 to C49, C48 to C50, C49 to C51, C50 to C52, C51 to C53, C52 to C54, C53 to C55, C54 to C56, C55 to C57, C56 to C58, C57 to C59
Connections:
- net GND: now also C43.2
- net at C42.1, D6.2 (A), Q5.3 (E)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: now also C43.1
Other:
- moved on the sheet: C42
