File: hardware/ADC7177B1/Power.kicad_sch (KiCad schematic)
At the start: 72 parts, among them J3 1715721, Q1 SI5618A, Q2 MMBT3904, Q3 FZT851, Q4 FZT951, Q5 FZT851, U10 TPS7A4901DGN, U4 THN 15-2425, U5 TEC 3-2419WI, U6 TPS7A4901DGN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

Commit message: Schematic changes
Parts:
- C28, C29, C30, C31, C32, C33, C34, C35, C36, C37, C38, C39, C40, C41, C42, C43, C52, C53, C54, C55, C56, C59: footprint Capacitor_SMD:C_1206_3216Metric_Pad1.33x1.80mm_HandSolder -> Capacitor_SMD:C_1206_3216Metric
- C44, C45, C46, C47, C48, C49, C50, C51, C57, C58: footprint Capacitor_SMD:C_0603_1608Metric_Pad1.08x0.95mm_HandSolder -> Capacitor_SMD:C_0603_1608Metric
Other:
- moved on the sheet: D2, R13
