File: hardware/ADC7177B1/ADC7177B1.kicad_pcb (KiCad board)
At the start: 2 copper layers, 55 parts, among them J1 20021111-00010T4LF, J2 RJ45_Wuerth_7499010121A, U1 STM32H743VITx, U2 24LC08B-E/MS, U3 LAN8742A, U5 TPS7A4901DGN, U6 ADC7177M1, U7 TPS7A3001DGN

Commit message: Schematic and PCB
Parts:
- added K1: SILxx-1Axx-71x, Relay_THT:Relay_SPST_StandexMeder_SIL_Form1A, F.Cu at (91.8, 76.3)
- added K2: SILxx-1Axx-71x, Relay_THT:Relay_SPST_StandexMeder_SIL_Form1A, F.Cu at (91.8, 83.0)
- added RN5: 1776-C68xx, ADC7177B1:1776-C68xx, F.Cu at (103.9, 65.7)
- added RN6: 1776-C68xx, ADC7177B1:1776-C68xx, F.Cu at (103.9, 70.6)
- added U8: AD8599ARZ, Package_SO:SOIC-8_3.9x4.9mm_P1.27mm, F.Cu at (114.5, 95.6)

Commit message: Schematic
Parts:
- removed K1, K2: SILxx-1Axx-71x, Relay_THT:Relay_SPST_StandexMeder_SIL_Form1A
- added C37: 10n, Capacitor_SMD:C_0603_1608Metric_Pad1.08x0.95mm_HandSolder, F.Cu at (21.1, 73.6)
- added C38: 10n, Capacitor_SMD:C_0603_1608Metric_Pad1.08x0.95mm_HandSolder, F.Cu at (21.1, 76.1)
- added C39: 10n, Capacitor_SMD:C_0603_1608Metric_Pad1.08x0.95mm_HandSolder, F.Cu at (21.1, 78.6)
- added C40: 10n, Capacitor_SMD:C_0603_1608Metric_Pad1.08x0.95mm_HandSolder, F.Cu at (21.1, 81.1)
- added R12: 1k, Resistor_SMD:R_0603_1608Metric_Pad0.98x0.95mm_HandSolder, F.Cu at (25.5, 73.6)
- added R13: 1k, Resistor_SMD:R_0603_1608Metric_Pad0.98x0.95mm_HandSolder, F.Cu at (25.5, 76.1)
- added R14: 1k, Resistor_SMD:R_0603_1608Metric_Pad0.98x0.95mm_HandSolder, F.Cu at (25.5, 78.6)
- added R15: 1k, Resistor_SMD:R_0603_1608Metric_Pad0.98x0.95mm_HandSolder, F.Cu at (25.5, 81.1)
- added R16: 120k, Resistor_SMD:R_0603_1608Metric_Pad0.98x0.95mm_HandSolder, F.Cu at (29.8, 73.6)
- added R17: 10k, Resistor_SMD:R_0603_1608Metric_Pad0.98x0.95mm_HandSolder, F.Cu at (29.8, 76.1)
- added R18: 120k, Resistor_SMD:R_0603_1608Metric_Pad0.98x0.95mm_HandSolder, F.Cu at (29.8, 78.6)
- added R19: 10k, Resistor_SMD:R_0603_1608Metric_Pad0.98x0.95mm_HandSolder, F.Cu at (29.8, 81.1)
- added R20: 2M2/0.05%, Resistor_SMD:R_1206_3216Metric_Pad1.30x1.75mm_HandSolder, F.Cu at (21.9, 47.5)
- added R21: 2M2/0.05%, Resistor_SMD:R_1206_3216Metric_Pad1.30x1.75mm_HandSolder, F.Cu at (21.9, 50.8)
- added R22: 2M2/0.05%, Resistor_SMD:R_1206_3216Metric_Pad1.30x1.75mm_HandSolder, F.Cu at (21.9, 54.1)
- added R23: 2M2/0.05%, Resistor_SMD:R_1206_3216Metric_Pad1.30x1.75mm_HandSolder, F.Cu at (21.9, 57.4)
- added R24: 2M2/0.05%, Resistor_SMD:R_1206_3216Metric_Pad1.30x1.75mm_HandSolder, F.Cu at (27.9, 47.5)
- added R25: 2M2/0.05%, Resistor_SMD:R_1206_3216Metric_Pad1.30x1.75mm_HandSolder, F.Cu at (27.9, 50.8)
- added R26: 2M2/0.05%, Resistor_SMD:R_1206_3216Metric_Pad1.30x1.75mm_HandSolder, F.Cu at (27.9, 54.1)
- added R27: 2M2/0.05%, Resistor_SMD:R_1206_3216Metric_Pad1.30x1.75mm_HandSolder, F.Cu at (27.9, 57.4)
- added R28: 1M1/0.05%, Resistor_SMD:R_1206_3216Metric_Pad1.30x1.75mm_HandSolder, F.Cu at (33.8, 47.5)
- added R29: 1M1/0.05%, Resistor_SMD:R_1206_3216Metric_Pad1.30x1.75mm_HandSolder, F.Cu at (33.8, 50.8)
- added R30: 100k/0.05%, Resistor_SMD:R_1206_3216Metric_Pad1.30x1.75mm_HandSolder, F.Cu at (33.8, 54.1)
- added R31: 100k/0.05%, Resistor_SMD:R_1206_3216Metric_Pad1.30x1.75mm_HandSolder, F.Cu at (33.8, 57.4)
- added R32: 510, Resistor_SMD:R_0603_1608Metric_Pad0.98x0.95mm_HandSolder, F.Cu at (21.1, 60.3)
- added R33: 510, Resistor_SMD:R_0603_1608Metric_Pad0.98x0.95mm_HandSolder, F.Cu at (21.1, 62.8)
- added R34: 1k2, Resistor_SMD:R_0603_1608Metric_Pad0.98x0.95mm_HandSolder, F.Cu at (21.1, 65.3)
- added R35: 10k/0.1%, Resistor_SMD:R_0603_1608Metric_Pad0.98x0.95mm_HandSolder, F.Cu at (21.1, 67.8)
- added R36: DNP, Resistor_SMD:R_0603_1608Metric_Pad0.98x0.95mm_HandSolder, F.Cu at (25.5, 60.3)
- added R37: 10k/0.1%, Resistor_SMD:R_0603_1608Metric_Pad0.98x0.95mm_HandSolder, F.Cu at (25.5, 62.8)
- added R38: 1100/0.1%, Resistor_SMD:R_0603_1608Metric_Pad0.98x0.95mm_HandSolder, F.Cu at (25.5, 65.3)
- added R39: 10k/0.1%, Resistor_SMD:R_0603_1608Metric_Pad0.98x0.95mm_HandSolder, F.Cu at (25.5, 67.8)
- added R40: 10k/0.1%, Resistor_SMD:R_0603_1608Metric_Pad0.98x0.95mm_HandSolder, F.Cu at (29.8, 60.3)
- added R41: 1k2, Resistor_SMD:R_0603_1608Metric_Pad0.98x0.95mm_HandSolder, F.Cu at (29.8, 62.8)
- added R42: 1k2, Resistor_SMD:R_0603_1608Metric_Pad0.98x0.95mm_HandSolder, F.Cu at (29.8, 65.3)
- added R43: 110/0.05%, Resistor_SMD:R_0603_1608Metric_Pad0.98x0.95mm_HandSolder, F.Cu at (29.8, 67.8)
- added U10: CPC1002N, Package_SO:SOP-4_3.8x4.1mm_P2.54mm, F.Cu at (53.0, 45.8)
- added U9: CPC1002N, Package_SO:SOP-4_3.8x4.1mm_P2.54mm, F.Cu at (36.2, 61.9)
- moved C1 121.8 mm to (52.5, 109.0)
- moved C10 121.8 mm to (56.9, 114.0)
- moved C11 121.8 mm to (56.9, 116.5)
- moved C12 121.8 mm to (56.9, 119.0)
- moved C13 121.8 mm to (56.9, 121.5)
- moved C14 121.8 mm to (56.9, 124.0)
- moved C2 121.8 mm to (52.5, 111.5)
- moved C3 121.8 mm to (52.5, 114.0)
- moved C4 121.8 mm to (52.5, 116.5)
- moved C5 121.8 mm to (52.5, 119.0)
- moved C6 121.8 mm to (52.5, 121.5)
- moved C7 121.8 mm to (52.5, 124.0)
- moved C8 121.8 mm to (56.9, 109.0)
- moved C9 121.8 mm to (56.9, 111.5)
- moved U5 121.8 mm to (35.5, 138.1)
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- renumbered U7 to U6, U6 to U7
Other:
- board outline added: 160 x 100 mm

Commit message: PCB
Parts:
- moved C40 170.7 mm to (187.2, 120.7), turned to 90 degrees
- moved C39 168.9 mm to (184.7, 120.7), turned to 90 degrees
- moved C38 167.1 mm to (182.2, 120.7), turned to 90 degrees
- moved R15 165.5 mm to (187.2, 116.4), turned to 90 degrees
- moved C37 165.4 mm to (179.7, 120.7), turned to 90 degrees
- moved R14 163.6 mm to (184.7, 116.4), turned to 90 degrees
- moved R13 161.8 mm to (182.2, 116.4), turned to 90 degrees
- moved R35 161.7 mm to (173.9, 120.7), turned to 90 degrees
- moved R19 160.4 mm to (187.2, 112.0), turned to 90 degrees
- moved R34 160.1 mm to (171.4, 120.7), turned to 90 degrees
- moved R12 160.0 mm to (179.7, 116.4), turned to 90 degrees
- moved R33 158.7 mm to (168.9, 120.7), turned to 90 degrees
- moved R18 158.4 mm to (184.7, 112.0), turned to 90 degrees
- moved U10 157.3 mm to (197.5, 107.9)
- moved U8 157.3 mm to (199.1, 119.5)
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
Commit message: PCB
Parts:
- added C27: 10u/50V, Capacitor_SMD:C_1206_3216Metric_Pad1.33x1.80mm_HandSolder, F.Cu at (43.7, 139.0)
- added C28: 10u/50V, Capacitor_SMD:C_1206_3216Metric_Pad1.33x1.80mm_HandSolder, F.Cu at (43.7, 142.3)
- added C29: 10u/50V, Capacitor_SMD:C_1206_3216Metric_Pad1.33x1.80mm_HandSolder, F.Cu at (105.1, 158.2)
- added C30: 10u/50V, Capacitor_SMD:C_1206_3216Metric_Pad1.33x1.80mm_HandSolder, F.Cu at (43.7, 145.7)
- added C31: 10u/50V, Capacitor_SMD:C_1206_3216Metric_Pad1.33x1.80mm_HandSolder, F.Cu at (43.7, 149.0)
- added C32: 10u/50V, Capacitor_SMD:C_1206_3216Metric_Pad1.33x1.80mm_HandSolder, F.Cu at (105.1, 161.5)
- added C33: 10u/50V, Capacitor_SMD:C_1206_3216Metric_Pad1.33x1.80mm_HandSolder, F.Cu at (49.7, 139.0)
- added C34: 10u/50V, Capacitor_SMD:C_1206_3216Metric_Pad1.33x1.80mm_HandSolder, F.Cu at (49.7, 142.3)
- added C35: 10u/50V, Capacitor_SMD:C_1206_3216Metric_Pad1.33x1.80mm_HandSolder, F.Cu at (105.1, 164.9)
- added C36: 10u/50V, Capacitor_SMD:C_1206_3216Metric_Pad1.33x1.80mm_HandSolder, F.Cu at (49.7, 145.7)
- added C37: 10u/50V, Capacitor_SMD:C_1206_3216Metric_Pad1.33x1.80mm_HandSolder, F.Cu at (49.7, 149.0)
- added C38: 10u/50V, Capacitor_SMD:C_1206_3216Metric_Pad1.33x1.80mm_HandSolder, F.Cu at (105.1, 168.2)
- added C39: 10u/50V, Capacitor_SMD:C_1206_3216Metric_Pad1.33x1.80mm_HandSolder, F.Cu at (55.7, 139.0)
- added C40: 10u/50V, Capacitor_SMD:C_1206_3216Metric_Pad1.33x1.80mm_HandSolder, F.Cu at (55.7, 142.3)
- added C41: 10u/50V, Capacitor_SMD:C_1206_3216Metric_Pad1.33x1.80mm_HandSolder, F.Cu at (105.1, 171.6)
- added C44: 10n, Capacitor_SMD:C_0603_1608Metric_Pad1.08x0.95mm_HandSolder, F.Cu at (104.3, 174.5)
- added C45: 10n, Capacitor_SMD:C_0603_1608Metric_Pad1.08x0.95mm_HandSolder, F.Cu at (104.3, 179.5)
- added C48: 10n, Capacitor_SMD:C_0603_1608Metric_Pad1.08x0.95mm_HandSolder, F.Cu at (104.3, 177.0)
- added C49: 10n, Capacitor_SMD:C_0603_1608Metric_Pad1.08x0.95mm_HandSolder, F.Cu at (104.3, 182.0)
- added C50: 10u/50V, Capacitor_SMD:C_1206_3216Metric_Pad1.33x1.80mm_HandSolder, F.Cu at (55.7, 145.7)
- added C51: 10u/50V, Capacitor_SMD:C_1206_3216Metric_Pad1.33x1.80mm_HandSolder, F.Cu at (55.7, 149.0)
- added C52: 10u/50V, Capacitor_SMD:C_1206_3216Metric_Pad1.33x1.80mm_HandSolder, F.Cu at (111.1, 158.2)
- added C53: 10u/50V, Capacitor_SMD:C_1206_3216Metric_Pad1.33x1.80mm_HandSolder, F.Cu at (117.1, 161.5)
- added C54: 10u/50V, Capacitor_SMD:C_1206_3216Metric_Pad1.33x1.80mm_HandSolder, F.Cu at (95.5, 175.4)
- added C55: 10n, Capacitor_SMD:C_0603_1608Metric_Pad1.08x0.95mm_HandSolder, F.Cu at (104.3, 184.6)
- added C56: 10n, Capacitor_SMD:C_0603_1608Metric_Pad1.08x0.95mm_HandSolder, F.Cu at (104.3, 187.1)
- added C57: 10u/50V, Capacitor_SMD:C_1206_3216Metric_Pad1.33x1.80mm_HandSolder, F.Cu at (117.1, 164.9)
- added C58: 0.1u, Capacitor_SMD:C_0603_1608Metric_Pad1.08x0.95mm_HandSolder, F.Cu at (89.9, 159.9)
- added C59: 0.1u, Capacitor_SMD:C_0603_1608Metric_Pad1.08x0.95mm_HandSolder, F.Cu at (89.9, 162.4)
- added C60: 0.1u, Capacitor_SMD:C_0603_1608Metric_Pad1.08x0.95mm_HandSolder, F.Cu at (41.5, 88.6)
- added C61: 0.1u, Capacitor_SMD:C_0603_1608Metric_Pad1.08x0.95mm_HandSolder, F.Cu at (41.5, 91.1)
- added C62: 0.1u, Capacitor_SMD:C_0603_1608Metric_Pad1.08x0.95mm_HandSolder, F.Cu at (67.1, 57.6)
- added C63: 0.1u, Capacitor_SMD:C_0603_1608Metric_Pad1.08x0.95mm_HandSolder, F.Cu at (67.1, 60.1)
- added C64: 0.1u, Capacitor_SMD:C_0603_1608Metric_Pad1.08x0.95mm_HandSolder, F.Cu at (67.1, 62.7)
- added C65: 0.1u, Capacitor_SMD:C_0603_1608Metric_Pad1.08x0.95mm_HandSolder, F.Cu at (67.1, 65.2)
- added D2: BZX84C10LT1G, Package_TO_SOT_SMD:SOT-23, F.Cu at (231.6, 102.0)
- added D3: 1N4148W, Diode_SMD:D_SOD-123, F.Cu at (255.0, 110.0)
- added D6: SS16, Diode_SMD:D_SMA, F.Cu at (126.5, 175.5)
- added D7: 1N4148W, Diode_SMD:D_SOD-123, F.Cu at (65.0, 121.9)
- added D8: 1N4148W, Diode_SMD:D_SOD-123, F.Cu at (65.0, 118.5)
- added H1: MountingHole, MountingHole:MountingHole_3.2mm_M3_DIN965_Pad, F.Cu at (84.0, 55.0)
- added H2: MountingHole, MountingHole:MountingHole_3.2mm_M3_DIN965_Pad, F.Cu at (84.0, 147.0)
- added H3: MountingHole, MountingHole:MountingHole_3.2mm_M3_DIN965_Pad, F.Cu at (236.0, 55.0)
- added H4: MountingHole, MountingHole:MountingHole_3.2mm_M3_DIN965_Pad, F.Cu at (236.0, 147.0)
- added J3: 1715721, TerminalBlock_Phoenix:TerminalBlock_Phoenix_MKDS-1,5-2_1x02_P5.00mm_Horizontal, F.Cu at (234.9, 95.2)
- added J4: Conn_01x01, ADC7177B1:S16N-PC, F.Cu at (94.4, 69.1)
- added J5: Conn_01x01, ADC7177B1:S16N-PC, F.Cu at (94.5, 88.5)
- added J6: Conn_01x01, ADC7177B1:S16N-PC, F.Cu at (94.3, 133.9)
- added J7: Conn_01x01, ADC7177B1:S16N-PC, F.Cu at (94.6, 113.2)
- added K1: G6SK-2F-DC5, ADC7177B1:G6SK-2F, F.Cu at (132.2, 72.9)
- added Q1: SI5618A, Package_TO_SOT_SMD:SOT-23, F.Cu at (237.0, 101.9)
- added Q2: MMBT3904, Package_TO_SOT_SMD:SOT-23, F.Cu at (249.6, 116.7)
- added Q3: FZT851, Package_TO_SOT_SMD:SOT-223, F.Cu at (120.0, 121.4)
- added Q4: FZT951, Package_TO_SOT_SMD:SOT-223, F.Cu at (80.8, 171.2)
- added Q5: FZT851, Package_TO_SOT_SMD:SOT-223, F.Cu at (125.0, 160.7)
- added Q6: MMBT3904, Package_TO_SOT_SMD:SOT-23, F.Cu at (64.6, 114.6)
- added Q7: MMBT3904, Package_TO_SOT_SMD:SOT-23, F.Cu at (64.6, 110.0)
- added R12: 0, Resistor_SMD:R_1206_3216Metric_Pad1.30x1.75mm_HandSolder, F.Cu at (255.0, 106.7)
- added R13: 100k, Resistor_SMD:R_0603_1608Metric_Pad0.98x0.95mm_HandSolder, F.Cu at (254.2, 112.9)
- added R14: 100k, Resistor_SMD:R_0603_1608Metric_Pad0.98x0.95mm_HandSolder, F.Cu at (254.2, 115.4)
- added R17: 1k, Resistor_SMD:R_0603_1608Metric_Pad0.98x0.95mm_HandSolder, F.Cu at (108.6, 174.5)
- added R20: 1k, Resistor_SMD:R_0603_1608Metric_Pad0.98x0.95mm_HandSolder, F.Cu at (108.6, 177.0)
- added R25: 120k, Resistor_SMD:R_0603_1608Metric_Pad0.98x0.95mm_HandSolder, F.Cu at (108.6, 179.5)
- added R26: 10k, Resistor_SMD:R_0603_1608Metric_Pad0.98x0.95mm_HandSolder, F.Cu at (108.6, 182.0)
- added R27: 120k, Resistor_SMD:R_0603_1608Metric_Pad0.98x0.95mm_HandSolder, F.Cu at (113.0, 174.5)
- added R28: 10k, Resistor_SMD:R_0603_1608Metric_Pad0.98x0.95mm_HandSolder, F.Cu at (113.0, 177.0)
- added R29: 120k, Resistor_SMD:R_0603_1608Metric_Pad0.98x0.95mm_HandSolder, F.Cu at (113.0, 179.5)
- added R30: 10k, Resistor_SMD:R_0603_1608Metric_Pad0.98x0.95mm_HandSolder, F.Cu at (113.0, 182.0)
- added R50: 510, Resistor_SMD:R_0603_1608Metric_Pad0.98x0.95mm_HandSolder, F.Cu at (41.5, 98.7)
- added R51: 510, Resistor_SMD:R_0603_1608Metric_Pad0.98x0.95mm_HandSolder, F.Cu at (41.5, 101.2)
- added R56: 510, Resistor_SMD:R_0603_1608Metric_Pad0.98x0.95mm_HandSolder, F.Cu at (41.5, 93.6)
- added R58: 510, Resistor_SMD:R_0603_1608Metric_Pad0.98x0.95mm_HandSolder, F.Cu at (41.5, 96.1)
- added R59: 10k, Resistor_SMD:R_0603_1608Metric_Pad0.98x0.95mm_HandSolder, F.Cu at (64.3, 127.3)
- added R60: 10k, Resistor_SMD:R_0603_1608Metric_Pad0.98x0.95mm_HandSolder, F.Cu at (64.3, 124.8)
- added R61: 510, Resistor_SMD:R_0603_1608Metric_Pad0.98x0.95mm_HandSolder, F.Cu at (67.1, 67.7)
- added R62: 510, Resistor_SMD:R_0603_1608Metric_Pad0.98x0.95mm_HandSolder, F.Cu at (67.1, 70.2)
- added U10: TPS7A4901DGN, Package_SO:HVSSOP-8-1EP_3x3mm_P0.65mm_EP1.57x1.89mm_ThermalVias, F.Cu at (118.8, 184.9)
- added U13: AD8599ARZ, Package_SO:SOIC-8_3.9x4.9mm_P1.27mm, F.Cu at (47.9, 90.7)
- added U4: THN 15-2425, ADC7177B1:THN_15-2425, F.Cu at (223.4, 72.6)
- added U5: TEC 3-2419WI, Converter_DCDC:Converter_DCDC_TRACO_TEC3-24xxUI_THT, F.Cu at (235.7, 113.5)
- added U8: TPS7A4901DGN, Package_SO:HVSSOP-8-1EP_3x3mm_P0.65mm_EP1.57x1.89mm_ThermalVias, F.Cu at (184.9, 111.9)
- added U9: TPS7A4901DGN, Package_SO:HVSSOP-8-1EP_3x3mm_P0.65mm_EP1.57x1.89mm_ThermalVias, F.Cu at (118.8, 180.3)
- added Y1: NX5032GA-16, ADC7177B1:NX5032GA, F.Cu at (64.4, 146.3)
- added Y2: NX5032GA-25, ADC7177B1:NX5032GA, F.Cu at (64.4, 139.6)
- moved C42 129.9 mm to (70.4, 191.1)
- moved C43 129.9 mm to (73.0, 191.1)
- moved C46 129.9 mm to (75.5, 191.1)
- moved C47 129.9 mm to (78.0, 191.1)
- moved R15 129.9 mm to (70.4, 186.7)
- moved R16 129.9 mm to (73.0, 186.7)
- moved R18 129.9 mm to (75.5, 186.7)
- moved R19 129.9 mm to (78.0, 186.7)
- moved R21 129.9 mm to (70.4, 182.4)
- moved R22 129.9 mm to (73.0, 182.4)
- moved R23 129.9 mm to (75.5, 182.4)
- moved R24 129.9 mm to (78.0, 182.4)
- moved R32 129.9 mm to (47.6, 190.3)
- moved R33 129.9 mm to (50.9, 190.3)
- moved R34 129.9 mm to (54.2, 190.3)
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- renumbered C37 to C42, C38 to C43, C39 to C46, C40 to C47, C7 to C6, C8 to C7, C6 to C8, D2 to D4, D3 to D5, R12 to R15, R13 to R16, R14 to R18, R15 to R19, R16 to R21, R17 to R22, R18 to R23, R19 to R24, R20 to R31, R21 to R32, R22 to R33, R23 to R34, R24 to R35, R25 to R36, R26 to R37, R27 to R38, R28 to R39, R29 to R40, R30 to R41, R31 to R42, R32 to R43, R33 to R44, R34 to R45, R35 to R46, R36 to R47, R37 to R48, R38 to R49, R39 to R52, R40 to R53, R41 to R54, R42 to R55, R43 to R57, U7 to U11, U8 to U12, U9 to U14, U10 to U15, U5 to U6, U6 to U7
Connections:
- net /Schematic/Frontend/MCU_Gx10 renamed /Schematic/Frontend/Gx10
- net /Schematic/Frontend/MCU_Gx100 renamed /Schematic/Frontend/Gx100

Commit message: PCB
Parts:
- added C43: 10u/50V, Capacitor_SMD:C_1206_3216Metric_Pad1.33x1.80mm_HandSolder, F.Cu at (176.7, 106.2)
- added C8: 0.1u, Capacitor_SMD:C_0603_1608Metric_Pad1.08x0.95mm_HandSolder, B.Cu at (193.8, 139.6)
- added L1: 74408943100, ADC7177B1:74408943100, F.Cu at (207.1, 65.5)
- added L2: 74408943100, ADC7177B1:74408943100, F.Cu at (206.9, 80.9)
- added L3: 74408943100, ADC7177B1:74408943100, F.Cu at (218.4, 102.6)
- C10: renamed from C8; moved to B.Cu
- C11: renamed from C10; moved to B.Cu
- C12: renamed from C11; moved to B.Cu
- C5, C6, FB1, RN3, RN4: moved to B.Cu
- R51: renamed from R49; value 1100/0.1% -> 1k1/0.1%
- moved RN4 215.3 mm to (225.6, 134.7)
- moved D4 200.6 mm to (192.7, 65.8), turned to -90 degrees
- moved D5 194.0 mm to (192.8, 81.9), turned to 90 degrees
- moved C28 181.4 mm to (207.4, 60.8)
- moved C31 180.0 mm to (207.1, 70.4)
- moved D1 179.4 mm to (194.9, 122.9), turned to 180 degrees
- moved C32 178.7 mm to (206.9, 76.3)
- moved FB1 176.6 mm to (196.0, 143.8)
- moved R15 175.3 mm to (192.9, 61.2), turned to 180 degrees
- moved R18 174.2 mm to (196.3, 61.2), turned to 0 degrees
- moved C37 173.5 mm to (201.0, 60.8)
- moved C29 172.8 mm to (206.9, 85.5)
- moved RN1 170.4 mm to (190.5, 122.9), turned to 90 degrees
- moved R16 168.6 mm to (200.4, 76.3), turned to 0 degrees
- moved U7 164.8 mm to (160.4, 97.7)
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- renumbered C12 to C13, C13 to C14, C14 to C15, C15 to C16, C16 to C17, C17 to C18, C18 to C19, C19 to C20, C20 to C21, C21 to C22, C22 to C23, C23 to C24, C24 to C25, C25 to C26, C26 to C27, C27 to C28, C28 to C29, C29 to C30, C30 to C31, C31 to C32, C32 to C33, C33 to C34, C34 to C35, C35 to C36, C36 to C37, C37 to C38, C38 to C39, C39 to C40, C40 to C41, C41 to C42, C42 to C44, C43 to C45, C44 to C46, C45 to C47, C46 to C48, C47 to C49, C48 to C50, C49 to C51, C50 to C52, C51 to C53, C52 to C54, C53 to C55, C54 to C56, C55 to C57, C56 to C58, C57 to C59, C58 to C60, C59 to C61, C60 to C62, C61 to C63, C65 to C64, C64 to C65, C62 to C66, C63 to C67, R61 to R45, R62 to R46, R45 to R47, R46 to R48, R47 to R49, R48 to R50, R50 to R52, R51 to R53, R52 to R54, R53 to R55, R54 to R56, R55 to R57, R56 to R58, R57 to R59, R58 to R60, R59 to R61, R60 to R62
Connections:
- U1 pad 20: +3.3VADC -> +3.3V

Commit message: PCB
Parts:
- C10: moved to F.Cu
- C17, C18, C20, C21, C24, C25, C26, C27, D2, D3, D7, D8, Q1, Q2, Q6, Q7, R10, R11, R12, R6, R61, R62, R8: moved to B.Cu
- moved R32 115.2 mm to (103.5, 89.5), turned to 0 degrees
- moved R36 114.3 mm to (111.5, 89.5), turned to 0 degrees
- moved R40 114.3 mm to (119.5, 89.5), turned to 0 degrees
- moved R34 112.0 mm to (107.6, 91.8), turned to 0 degrees
- moved C56 111.6 mm to (186.9, 111.5), turned to 90 degrees
- moved R38 111.0 mm to (115.6, 91.8), turned to 0 degrees
- moved R42 110.9 mm to (123.6, 91.8), turned to 180 degrees
- moved C57 107.8 mm to (186.9, 115.4)
- moved C58 103.8 mm to (176.5, 112.5), turned to -90 degrees
- moved R29 93.4 mm to (178.1, 112.5), turned to -90 degrees
- moved R30 93.0 mm to (177.3, 114.9)
- moved C59 85.1 mm to (182.1, 110.0)
- moved C27 70.6 mm to (222.6, 128.0), turned to 90 degrees
- moved C19 64.0 mm to (211.6, 127.3), turned to 90 degrees
- moved C26 62.1 mm to (217.6, 133.9), turned to 90 degrees
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Connections:
- U1 pad 64: /Schematic/MCU/LED_RED -> /Schematic/MCU/LED_GREEN
- U1 pad 65: /Schematic/MCU/LED_GREEN -> /Schematic/MCU/LED_RED
Routing:
- net Net-(K1-Pad8): track 0.00 -> 30.4 mm, vias 0 -> 2
- net Net-(K1-Pad3): track 0.00 -> 28.9 mm
- net Net-(K1-Pad10): track 0.00 -> 28.5 mm
- net Net-(J6-Pin_1): track 0.00 -> 26.6 mm
- net Net-(J7-Pin_1): track 0.00 -> 26.2 mm
- net Net-(K1-Pad5): track 0.00 -> 24.4 mm, vias 0 -> 2
- net /Schematic/ADC Module/IN-: track 0.00 -> 21.2 mm
- net /Schematic/ADC Module/IN+: track 0.00 -> 20.9 mm
- net Net-(RN6-R2): track 0.00 -> 17.5 mm
- net Net-(U12B--): track 0.00 -> 16.1 mm
- net +3.3V: track 0.00 -> 15.7 mm, vias 0 -> 9
- net Net-(RN5-R2): track 0.00 -> 15.7 mm
- net Net-(J4-Pin_1): track 0.00 -> 14.5 mm
- net Net-(J5-Pin_1): track 0.00 -> 14.2 mm
- net Net-(U12A--): track 0.00 -> 13.0 mm
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Other:
- copper layers 2 -> 4
