File: hardware/ADC7177B1/MCU.kicad_sch (KiCad schematic)
At the start: 27 parts, among them J1 20021111-00010T4LF, U1 STM32H743VITx, U2 24LC08B-E/MS, Y1 NX5032GA-16

Commit message: PCB
Parts:
- Y1: footprint ETH1HMSR-SMS:NX5032GA -> ADC7177B1:NX5032GA
- renumbered C7 to C6, C8 to C7, C6 to C8
Other:
- moved on the sheet: C1, C10, C11, C12, C13, C2, C3, C4, C5, C6, C7, C8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

Commit message: PCB
Parts:
- added C8: 0.1u, Capacitor_SMD:C_0603_1608Metric_Pad1.08x0.95mm_HandSolder, symbol Device:C
- renumbered C8 to C10, C10 to C11, C11 to C12, C12 to C13, C13 to C14, C14 to C15
Connections:
- net +3.3VADC is gone; now on net +3.3V: U1.20 (VREF+)
- net +3.3V: now also C8.1
- net GND: now also C8.2
Other:
- moved on the sheet: C10, C13, C14, FB1

Commit message: PCB
Connections:
- net LED_GREEN: now also U1.64 (PC7); no longer U1.65 (PC8)
- net LED_RED: now also U1.65 (PC8); no longer U1.64 (PC7)
Changed lines of the file:
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@@
 	)
 	(label "LED_GREEN"
-		(at 186.69 135.89 180)
+		(at 186.69 133.35 180)
 		(effects
 			(font
@@
 	)
 	(label "LED_RED"
-		(at 186.69 133.35 180)
+		(at 186.69 135.89 180)
 		(effects
 			(font
