File: hardware/ADC7177B1/ADC_Module.kicad_sch (KiCad schematic)
At the start: 1 part, among them U6 ADC7177M1

Commit message: PCB and schematic
Parts:
- U6: footprint (none) -> ADC7177B1:ADC7177M1
Changed lines of the file:
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@@
 			)
 		)
-		(property "Footprint" ""
+		(property "Footprint" "ADC7177B1:ADC7177M1"
 			(at 142.24 78.74 0)
 			(effects

Commit message: Schematic
Parts:
- renumbered U6 to U7
Changed lines of the file:
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@@
 		(dnp no)
 		(fields_autoplaced yes)
-		(property "Reference" "#PWR074"
+		(property "Reference" "#PWR078"
 			(at 124.46 115.57 0)
 			(effects
@@
 			(project ""
 				(path "/06a56fb9-779c-428e-b281-14ac9294755f/ce8ead21-c650-4940-b61e-074f59a08930/07044147-0e8a-4c72-a8b6-f4a6a6e21869"
-					(reference "#PWR074")
+					(reference "#PWR078")
 					(unit 1)
 				)
@@
 		(dnp no)
 		(fields_autoplaced yes)
-		(property "Reference" "#PWR075"
+		(property "Reference" "#PWR079"
 			(at 160.02 96.52 0)
 			(effects
@@
 			(project "ADC7177B1"
 				(path "/06a56fb9-779c-428e-b281-14ac9294755f/ce8ead21-c650-4940-b61e-074f59a08930/07044147-0e8a-4c72-a8b6-f4a6a6e21869"
-					(reference "#PWR075")
+					(reference "#PWR079")
 					(unit 1)
 				)
@@
 		(dnp no)
 		(fields_autoplaced yes)
-		(property "Reference" "#PWR077"
+		(property "Reference" "#PWR074"
 			(at 127 67.31 0)
 			(effects
@@
 			(project ""
 				(path "/06a56fb9-779c-428e-b281-14ac9294755f/ce8ead21-c650-4940-b61e-074f59a08930/07044147-0e8a-4c72-a8b6-f4a6a6e21869"
-					(reference "#PWR077")
+					(reference "#PWR074")
 					(unit 1)
 				)
@@
 		(dnp no)
 		(fields_autoplaced yes)
-		(property "Reference" "#PWR079"
+		(property "Reference" "#PWR077"
 			(at 127 88.9 0)
 			(effects
@@
 			(project ""
 				(path "/06a56fb9-779c-428e-b281-14ac9294755f/ce8ead21-c650-4940-b61e-074f59a08930/07044147-0e8a-4c72-a8b6-f4a6a6e21869"
-					(reference "#PWR079")
+					(reference "#PWR077")
 					(unit 1)
 				)
@@
 		(dnp no)
 		(fields_autoplaced yes)
-		(property "Reference" "#PWR076"
+		(property "Reference" "#PWR075"
 			(at 127 73.66 0)
 			(effects
@@
 			(project ""
 				(path "/06a56fb9-779c-428e-b281-14ac9294755f/ce8ead21-c650-4940-b61e-074f59a08930/07044147-0e8a-4c72-a8b6-f4a6a6e21869"
-					(reference "#PWR076")
+					(reference "#PWR075")
 					(unit 1)
 				)
@@
 		(dnp no)
 		(fields_autoplaced yes)
-		(property "Reference" "U6"
+		(property "Reference" "U7"
 			(at 142.24 41.91 0)
 			(effects
@@
 			(project ""
 				(path "/06a56fb9-779c-428e-b281-14ac9294755f/ce8ead21-c650-4940-b61e-074f59a08930/07044147-0e8a-4c72-a8b6-f4a6a6e21869"
-					(reference "U6")
+					(reference "U7")
 					(unit 1)
 				)
@@
 		(dnp no)
 		(fields_autoplaced yes)
-		(property "Reference" "#PWR078"
+		(property "Reference" "#PWR076"
 			(at 127 81.28 0)
 			(effects
@@
 			(project ""
 				(path "/06a56fb9-779c-428e-b281-14ac9294755f/ce8ead21-c650-4940-b61e-074f59a08930/07044147-0e8a-4c72-a8b6-f4a6a6e21869"
-					(reference "#PWR078")
-					(unit 1)
-				)
+					(reference "#PWR076")
+					(unit 1)
+				)

Commit message: PCB
Parts:
- renumbered U7 to U11
Other:
- note added: "2x FLE-108-01-G-DV-K-TR"
Changed lines of the file:
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@@
 	(generator_version "9.0")
 	(paper "A4")
+	(text "2x FLE-108-01-G-DV-K-TR"
+		(exclude_from_sim no)
+		(at 141.986 119.888 0)
+		(effects
+			(font
+				(size 1.27 1.27)
+			)
+		)
+	)
 	(junction
 		(at 124.46 102.87)
@@
 		(dnp no)
 		(fields_autoplaced yes)
-		(property "Reference" "#PWR078"
+		(property "Reference" "#PWR0106"
 			(at 124.46 115.57 0)
 			(effects
@@
 			(project ""
 				(path "/06a56fb9-779c-428e-b281-14ac9294755f/ce8ead21-c650-4940-b61e-074f59a08930/07044147-0e8a-4c72-a8b6-f4a6a6e21869"
-					(reference "#PWR078")
+					(reference "#PWR0106")
 					(unit 1)
 				)
@@
 		(dnp no)
 		(fields_autoplaced yes)
-		(property "Reference" "#PWR079"
+		(property "Reference" "#PWR0107"
 			(at 160.02 96.52 0)
 			(effects
@@
 			(project "ADC7177B1"
 				(path "/06a56fb9-779c-428e-b281-14ac9294755f/ce8ead21-c650-4940-b61e-074f59a08930/07044147-0e8a-4c72-a8b6-f4a6a6e21869"
-					(reference "#PWR079")
+					(reference "#PWR0107")
 					(unit 1)
 				)
@@
 		(dnp no)
 		(fields_autoplaced yes)
-		(property "Reference" "#PWR074"
+		(property "Reference" "#PWR0102"
 			(at 127 67.31 0)
 			(effects
@@
 			(project ""
 				(path "/06a56fb9-779c-428e-b281-14ac9294755f/ce8ead21-c650-4940-b61e-074f59a08930/07044147-0e8a-4c72-a8b6-f4a6a6e21869"
-					(reference "#PWR074")
+					(reference "#PWR0102")
 					(unit 1)
 				)
@@
 		(dnp no)
 		(fields_autoplaced yes)
-		(property "Reference" "#PWR077"
+		(property "Reference" "#PWR0105"
 			(at 127 88.9 0)
 			(effects
@@
 			(project ""
 				(path "/06a56fb9-779c-428e-b281-14ac9294755f/ce8ead21-c650-4940-b61e-074f59a08930/07044147-0e8a-4c72-a8b6-f4a6a6e21869"
-					(reference "#PWR077")
+					(reference "#PWR0105")
 					(unit 1)
 				)
@@
 		(dnp no)
 		(fields_autoplaced yes)
-		(property "Reference" "#PWR075"
+		(property "Reference" "#PWR0103"
 			(at 127 73.66 0)
 			(effects
@@
 			(project ""
 				(path "/06a56fb9-779c-428e-b281-14ac9294755f/ce8ead21-c650-4940-b61e-074f59a08930/07044147-0e8a-4c72-a8b6-f4a6a6e21869"
-					(reference "#PWR075")
+					(reference "#PWR0103")
 					(unit 1)
 				)
@@
 		(dnp no)
 		(fields_autoplaced yes)
-		(property "Reference" "U7"
+		(property "Reference" "U11"
 			(at 142.24 41.91 0)
 			(effects
@@
 			(project ""
 				(path "/06a56fb9-779c-428e-b281-14ac9294755f/ce8ead21-c650-4940-b61e-074f59a08930/07044147-0e8a-4c72-a8b6-f4a6a6e21869"
-					(reference "U7")
+					(reference "U11")
 					(unit 1)
 				)
@@
 		(dnp no)
 		(fields_autoplaced yes)
-		(property "Reference" "#PWR076"
+		(property "Reference" "#PWR0104"
 			(at 127 81.28 0)
 			(effects
@@
 			(project ""
 				(path "/06a56fb9-779c-428e-b281-14ac9294755f/ce8ead21-c650-4940-b61e-074f59a08930/07044147-0e8a-4c72-a8b6-f4a6a6e21869"
-					(reference "#PWR076")
+					(reference "#PWR0104")
 					(unit 1)
 				)
