File: hardware/ADC7177B1/Schematic.kicad_sch (KiCad schematic)
At the start: 0 parts

Commit message: Schematic and PCB
Other:
- added sheet Frontend (Frontend.kicad_sch)
Changed lines of the file:
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@@
+	)
+	(sheet
+		(at 52.07 41.91)
+		(size 26.67 36.83)
+		(exclude_from_sim no)
+		(in_bom yes)
+		(on_board yes)
+		(dnp no)
+		(fields_autoplaced yes)
+		(stroke
+			(width 0.1524)
+			(type solid)
+		)
+		(fill
+			(color 0 0 0 0.0000)
+		)
+		(property "Sheetname" "Frontend"
+			(at 52.07 41.1984 0)
+			(effects
+				(font
+					(size 1.27 1.27)
+				)
+				(justify left bottom)
+			)
+		)
+		(property "Sheetfile" "Frontend.kicad_sch"
+			(at 52.07 79.3246 0)
+			(effects
+				(font
+					(size 1.27 1.27)
+				)
+				(justify left top)
+			)
+		)
+		(instances
+			(project "ADC7177B1"
+				(path "/06a56fb9-779c-428e-b281-14ac9294755f/ce8ead21-c650-4940-b61e-074f59a08930"
+					(page "7")
+				)
+			)
+		)
 	)
 	(sheet

Commit message: Schematic
Other:
- note removed: "AD797"
Changed lines of the file:
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@@
 	(generator_version "9.0")
 	(paper "A4")
-	(text "AD797\n"
-		(exclude_from_sim no)
-		(at 83.566 53.848 0)
-		(effects
-			(font
-				(size 1.27 1.27)
-			)
-		)
-	)
 	(wire
 		(pts
@@
 	)
 	(sheet
-		(at 52.07 41.91)
+		(at 68.58 43.18)
 		(size 26.67 36.83)
 		(exclude_from_sim no)
@@
 		)
 		(property "Sheetname" "Frontend"
-			(at 52.07 41.1984 0)
+			(at 68.58 42.4684 0)
 			(effects
 				(font
@@
 		)
 		(property "Sheetfile" "Frontend.kicad_sch"
-			(at 52.07 79.3246 0)
-			(effects
-				(font
+			(at 68.58 80.5946 0)
+			(effects
+				(font

Commit message: PCB
Parts:
- added H1, H2, H3, H4: MountingHole, MountingHole:MountingHole_3.2mm_M3_DIN965_Pad, symbol Mechanical:MountingHole
Other:
- sheet Frontend ports: added Gx10, Gx100, IN+, IN-, RLY_R, RLY_S; removed none
- sheet MCU ports: added A0N, A0P, A1N, A1P, A2N, A2P, DIN, DOUT, Gx10, Gx100, IN_CPL, RLY_R, RLY_S, SCLK, ~{CS}, ~{SYNC}/~{ERR}; removed none

Commit message: PCB
Parts:
- added H5, H6, H7, H8: MountingHole, MountingHole:MountingHole_2.5mm_Pad_TopBottom, symbol Mechanical:MountingHole

Commit message: Schematic changes
Other:
- added sheet Reference (Reference.kicad_sch)
Changed lines of the file:
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@@
+	)
+	(sheet
+		(at 31.75 93.98)
+		(size 38.1 31.75)
+		(exclude_from_sim no)
+		(in_bom yes)
+		(on_board yes)
+		(dnp no)
+		(fields_autoplaced yes)
+		(stroke
+			(width 0.1524)
+			(type solid)
+		)
+		(fill
+			(color 0 0 0 0.0000)
+		)
+		(property "Sheetname" "Reference"
+			(at 31.75 93.2684 0)
+			(effects
+				(font
+					(size 1.27 1.27)
+				)
+				(justify left bottom)
+			)
+		)
+		(property "Sheetfile" "Reference.kicad_sch"
+			(at 31.75 126.3146 0)
+			(effects
+				(font
+					(size 1.27 1.27)
+				)
+				(justify left top)
+			)
+		)
+		(instances
+			(project "ADC7177B1"
+				(path "/06a56fb9-779c-428e-b281-14ac9294755f/ce8ead21-c650-4940-b61e-074f59a08930"
+					(page "10")
+				)
+			)
+		)
 	)
 	(sheet
